File: Hardware/AnalogFrontEnd/Amplifier.kicad_sch (KiCad schematic)
At the start: 0 parts

Commit message: add bias supply circuit
Parts:
- added D1: D_SiPM, symbol Device:D_SiPM
Changed lines of the file:
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@@
+		)
+	)
+	(symbol
+		(lib_id "Device:D_SiPM")
+		(at 106.68 110.49 270)
+		(unit 1)
+		(body_style 1)
+		(exclude_from_sim no)
+		(in_bom yes)
+		(on_board yes)
+		(in_pos_files yes)
+		(dnp no)
+		(fields_autoplaced yes)
+		(property "Reference" "D1"
+			(at 111.76 109.5374 90)
+			(show_name no)
+			(do_not_autoplace no)
+			(effects
+				(font
+					(size 1.27 1.27)
+				)
+				(justify left)
+			)
+		)
+		(property "Value" "D_SiPM"
+			(at 111.76 112.0774 90)
+			(show_name no)
+			(do_not_autoplace no)
+			(effects
+				(font
+					(size 1.27 1.27)
+				)
+				(justify left)
+			)
+		)
+		(property "Footprint" ""
+			(at 111.125 111.76 0)
+			(hide yes)
+			(show_name no)
+			(do_not_autoplace no)
+			(effects
+				(font
+					(size 1.27 1.27)
+				)
+			)
+		)
+		(property "Datasheet" ""
+			(at 106.68 110.49 0)
+			(hide yes)
+			(show_name no)
+			(do_not_autoplace no)
+			(effects
+				(font
+					(size 1.27 1.27)
+				)
+			)
+		)
+		(property "Description" "Silicon photomultiplier"
+			(at 106.68 110.49 0)
+			(hide yes)
+			(show_name no)
+			(do_not_autoplace no)
+			(effects
+				(font
+					(size 1.27 1.27)
+				)
+			)
+		)
+		(pin "2"
+		)
+		(pin "1"
+		)
+		(instances
+			(project "AnalogFrontEnd"
+				(path "/b3e88616-4405-48d6-aecf-2659499541fb/c173cbc7-a48e-44ee-8730-76995ac7089c"
+					(reference "D1")
+					(unit 1)
+				)
+			)
 		)
 	)

Commit message: add draft of data processing circuit
Changed lines of the file:
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@@
 	(generator_version "10.0")
 	(paper "A4")
-	(hierarchical_label "SIPM_PULSE_RAW"
+	(hierarchical_label "SIPM_ADC_N"
+		(shape output)
+		(at 138.43 142.24 0)
+		(effects
+			(font
+				(size 1.27 1.27)
+			)
+			(justify left)
+		)
+	)
+	(hierarchical_label "SIPM_ADC_P"
+		(shape output)
+		(at 121.92 134.62 0)
+		(effects
+			(font
+				(size 1.27 1.27)
+			)
+			(justify left)
+		)
+	)
+	(hierarchical_label "VEE_2V5"
 		(shape input)
-		(at 139.7 110.49 0)
+		(at 152.4 119.38 0)
 		(effects
 			(font
@@
 		(effects
 			(font
+				(size 1.27 1.27)
+			)
+			(justify left)
+		)
+	)
+	(hierarchical_label "VCC_2V5"
+		(shape input)
+		(at 153.67 132.08 0)
+		(effects
+			(font
