File: Hardware/ProcessingAndPower/ProcessingAndPower.kicad_sch (KiCad schematic)
At the start: 0 parts

Commit message: add draft of data processing circuit
Other:
- added sheet ADC (ADC.kicad_sch)
- added sheet ExternalCommunication (ExternalCommunication.kicad_sch)
- added sheet ExternalConnector (ExternalConnector.kicad_sch)
- added sheet FPGA (FPGA.kicad_sch)
- added sheet PowerSupply (PowerSupply.kicad_sch)
