File: Hardware/SiPMOverlightProtection.kicad_sch (KiCad schematic)
At the start: 0 parts

Commit message: fix: #145, fix: #159
Parts:
- added R22, R23, R24: TBD, Resistor_SMD:R_0805_2012Metric, symbol Device:R
Connections:
- net SIPM_BIAS: now also R24.2
- net SIPM_OVERLIGHT_FAULT: now also R23.2
- new net GND: R22.1, R23.1, R24.1
- new net SIPM_BIAS_REG: R22.2
Other:
- note added: "TODO: this sheet is empty but silence warnings hile working on other sheets"
- company: (none) -> RG
- title: (none) -> SiPM Over-Illumination Protection
