File: Hardware/FPGA.kicad_sch (KiCad schematic)
At the start: 1 part, among them U6 ICE40HX4K-TQ144

Commit message: fix: #145, fix: #159
Parts:
- added C34, C35, C36, C37, C38, C42, C43, C44, C46: 100n, Capacitor_SMD:C_0805_2012Metric, symbol Device:C
- added D2: LED, symbol Device:LED
- added R31, R63: 10k, Resistor_SMD:R_0805_2012Metric, symbol Device:R
- added R62: 100R, Resistor_SMD:R_0805_2012Metric, symbol Device:R
- added R64: 680R, Resistor_SMD:R_0805_2012Metric, symbol Device:R
- added SW1: SW_Push, symbol Switch:SW_Push
Connections:
- net OTR: now also U6.124 (IOT_191)
- net SIPM_ADC1: now also U6.110 (IOT_168)
- net SIPM_ADC10: now also U6.120 (IOT_179)
- net SIPM_ADC11: now also U6.121 (IOT_181)
- net SIPM_ADC12: now also U6.122 (IOT_190)
- net SIPM_ADC2: now also U6.112 (IOT_169)
- net SIPM_ADC3: now also U6.113 (IOT_170)
- net SIPM_ADC4: now also U6.114 (IOT_171)
- net SIPM_ADC5: now also U6.115 (IOT_172)
- net SIPM_ADC6: now also U6.116 (IOT_173)
- net SIPM_ADC7: now also U6.117 (IOT_174)
- net SIPM_ADC8: now also U6.118 (IOT_177)
- net SIPM_ADC9: now also U6.119 (IOT_178)
- net SIPM_EN: now also U6.125 (IOT_192)
- net SIPM_OVERLIGHT_FAULT: now also U6.128 (IOT_197_GBIN1)
- net VCC_1V2: now also U6.126 (VCCPLL1), U6.54 (VCCPLL0), C35.1, C42.1
- net VCC_3V3: now also U6.100 (VCCIO_1), U6.111 (VCC), U6.123 (VCCIO_0), U6.131 (VCCIO_0), U6.27 (VCC), U6.30 (VCCIO_3), U6.40 (VCC), U6.46 (VCCIO_2), U6.57 (VCCIO_2), U6.6 (VCCIO_3), U6.72 (VCC_SPI), U6.89 (VCCIO_1), U6.92 (VCC), C34.1, C36.1, C37.1, C38.1, C44.1, C46.1, R31.2, R63.2
- net GND: now reaches U6.103 (GND), U6.13 (GND), U6.132 (GND), U6.14 (GND), U6.140 (GND), U6.5 (GND), U6.59 (GND), U6.69 (GND), U6.86 (GND)
- net GND: now also U6.127 (GNDPLL1), U6.53 (GNDPLL0), C34.2, C35.2, C36.2, C37.2, C38.2, C42.2, C43.2, C44.2, C46.2, D2.1 (K), SW1.2
- net VCC_2V5: now reaches U6.108 (VPP_2V5)
- net VCC_2V5: now also C43.1
- net CFG_DONE: now reaches U6.65 (CDONE)
- net CFG_DONE: now also R63.1
- net at U6.66 (~{CRESET}): now also R31.1, R62.1, SW1.1
- net CFG_SPI_MOSI: now reaches U6.67 (IOB_105_SDO)
- net CFG_SPI_MISO: now reaches U6.68 (IOB_106_SDI)
- net CFG_SPI_SCK: now reaches U6.70 (IOB_107_SCK)
- net CFG_SPI_CS: now reaches U6.71 (IOB_108_SS)
- net at U6.144 (IOT_222): now also R64.2
- new net: D2.2 (A), R64.1
- new net CFG_RESET: R62.2
- no-connect marks 103 -> 88
Other:
- company: (none) -> RG
- title: (none) -> iCE40HX4K FPGA Core & I/O Banks
- moved on the sheet: U6A, U6B, U6C, U6D, U6E

Commit message: fix: #160, fix: #163, fix: #164
Parts:
- added R92, R93: 2k2, Resistor_SMD:R_0805_2012Metric, symbol Device:R
Connections:
- net SIPM_BIAS_I2C_SDA: now reaches U6.129 (IOT_198_GBIN0)
- net SIPM_BIAS_I2C_SDA: now also R93.2
- net SIPM_EN renamed SIPM_BIAS_OK
- net SIPM_OVERLIGHT_FAULT renamed SIPM_BIAS_I2C_SCL
- net SIPM_BIAS_I2C_SCL: now also R92.2
- net VCC_1V2 renamed +1V2_FPGA
- net VCC_2V5 renamed +2V5_FPGA
- net VCC_3V3 renamed +3V3_FPGA
- net +3V3_FPGA: now also R92.1, R93.1
- no-connect marks 88 -> 87
