File: Hardware/UserInterface.kicad_sch (KiCad schematic)
At the start: 0 parts

Commit message: fix: #145, fix: #159
Other:
- company: (none) -> RG
- title: (none) -> User Interface
Changed lines of the file:
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@@
 	(generator_version "10.0")
 	(paper "A4")
+	(title_block
+		(title "User Interface")
+		(date "2026-04-06")
+		(rev "1.0")
+		(company "RG")
+	)
 )
