File: Hardware/SiPMBias.kicad_sch (KiCad schematic)
At the start: 0 parts

Commit message: fix: #170, fix: #144, fix: #132
Other:
- sheet SiPMBiasControl ports: added +3V3_A; removed +2V5_A
Changed lines of the file:
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@@
-		)
-	)
-	(hierarchical_label "+2V5_A"
-		(shape input)
-		(at 73.66 45.72 180)
-		(effects
-			(font
-				(size 1.27 1.27)
-			)
-			(justify right)
 		)
 	)
@@
 			)
 			(justify left)
+		)
+	)
+	(hierarchical_label "+3V3_A"
+		(shape input)
+		(at 73.66 45.72 180)
+		(effects
+			(font
+				(size 1.27 1.27)
+			)
+			(justify right)
 		)
 	)
@@
 			(project "GammaSpectrometer"
 				(path "/d6192878-4721-4ef4-99ff-dbbad0502886/26c85e8f-d7e7-4def-9549-c7a26d210092"
-					(page "5")
+					(page "11")
 				)
 			)
@@
 			)
 		)
-		(pin "+2V5_A" input
-			(at 86.36 82.55 180)
-			(effects
-				(font
-					(size 1.27 1.27)
-				)
-				(justify left)
-			)
-		)
 		(pin "VBIAS_EN" output
 			(at 127 80.01 0)
@@
 		(pin "+3V3_D" input
 			(at 86.36 80.01 180)
+			(effects
+				(font
+					(size 1.27 1.27)
+				)
+				(justify left)
+			)
+		)
+		(pin "+3V3_A" input
+			(at 86.36 82.55 180)
 			(effects
 				(font
@@
 			(project "GammaSpectrometer"
 				(path "/d6192878-4721-4ef4-99ff-dbbad0502886/26c85e8f-d7e7-4def-9549-c7a26d210092"
-					(page "4")
+					(page "12")
 				)
 			)
@@
 			(project "GammaSpectrometer"
 				(path "/d6192878-4721-4ef4-99ff-dbbad0502886/26c85e8f-d7e7-4def-9549-c7a26d210092"
-					(page "16")
-				)
-			)
+					(page "13")
+				)
+			)
