File: Hardware/AFEChannel2.kicad_sch (KiCad schematic)
At the start: 30 parts, among them U2101 OPA690xDBV, U2102 AD8139

Commit message: fix: #170
Parts:
- U2102: symbol DataAcquisitionUnit:AD8139 -> GammaSpectrometer:AD8139
Changed lines of the file:
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@@
 	)
 	(symbol
-		(lib_id "DataAcquisitionUnit:AD8139")
+		(lib_id "GammaSpectrometer:AD8139")
 		(at 140.97 44.45 0)
 		(unit 1)
@@
 	)
 	(group "AFE single channel"
-		(lib_id "GammaSpectrometer:AFE single channel")
-		(members "1d95dfca-94b0-4310-b12d-53215fc9c938")
-	)
-	(group "AFE single channel"
