File: Hardware/ExternalConnector.kicad_sch (KiCad schematic)
At the start: 5 parts, among them J1 DE9_Pins_MountingHoles, J2 Conn_Coaxial, J3 Conn_Coaxial

Commit message: fix: #170, fix #144
Parts:
- TP20, TP21: footprint TestPoint:TestPoint_Pad_D1.5mm -> TestPoint:TestPoint_Pad_D1.0mm
Changed lines of the file:
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@@
 			)
 		)
-		(property "Footprint" "TestPoint:TestPoint_Pad_D1.5mm"
+		(property "Footprint" "TestPoint:TestPoint_Pad_D1.0mm"
 			(at 138.43 106.68 0)
 			(hide yes)
@@
 			)
 		)
-		(property "Footprint" "TestPoint:TestPoint_Pad_D1.5mm"
+		(property "Footprint" "TestPoint:TestPoint_Pad_D1.0mm"
 			(at 128.27 130.81 0)
 			(hide yes)
