File: Hardware/GammaSpectrometer.kicad_pcb (KiCad board)
At the start: 2 copper layers, 100 x 100 mm, 273 parts, among them U10 LT3093, U11 AP2112K-3.3, U12 AP2112K-1.2, U14 LT3042, U15 LT3042, U16 LT8330IS6, U17 NCP163ASN330T1G (3v3), U18 5PB1102PGGK, U2 REF3220AMDBVREP, U5 TPS7A4901, U6 ICE40HX4K-TQ144, U7 AP2112K-3.3, U7 LT8330IS6, U7 XLH736065.000000I, U8 AP2112K-1.2, U8 LT8330IS6, U9 LT3093

Commit message: fix: #145, fix: #159
Parts:
- added C34: 100n, Capacitor_SMD:C_0805_2012Metric, F.Cu at (95.3, 35.1)
- added C35: 100n, Capacitor_SMD:C_0805_2012Metric, F.Cu at (147.6, 18.3)
- added C35: 100n, Capacitor_SMD:C_0805_2012Metric, F.Cu at (95.3, 38.1)
- added C36: 100n, Capacitor_SMD:C_0805_2012Metric, F.Cu at (95.3, 41.1)
- added C37: 100n, Capacitor_SMD:C_0805_2012Metric, F.Cu at (95.3, 44.1)
- added C38: 100n, Capacitor_SMD:C_0805_2012Metric, F.Cu at (95.3, 47.1)
- added C42: 100n, Capacitor_SMD:C_0805_2012Metric, F.Cu at (147.6, 21.3)
- added C43: 100n, Capacitor_SMD:C_0805_2012Metric, F.Cu at (147.6, 24.3)
- added C44: 100n, Capacitor_SMD:C_0805_2012Metric, F.Cu at (147.6, 27.3)
- added C46: 100n, Capacitor_SMD:C_0805_2012Metric, F.Cu at (147.6, 30.3)
- added C98: 100n, Capacitor_SMD:C_0805_2012Metric, F.Cu at (162.9, 24.9)
- added C99: 10n, Capacitor_SMD:C_0805_2012Metric, F.Cu at (162.9, 28.0)
- added R22: TBD, Resistor_SMD:R_0805_2012Metric, F.Cu at (101.8, 35.0)
- added R23: TBD, Resistor_SMD:R_0805_2012Metric, F.Cu at (101.8, 38.0)
- added R24: TBD, Resistor_SMD:R_0805_2012Metric, F.Cu at (101.8, 40.9)
- added R29: TBD, Resistor_SMD:R_0805_2012Metric, F.Cu at (101.8, 45.9)
- added R30: TBD, Resistor_SMD:R_0805_2012Metric, F.Cu at (101.8, 48.8)
- added R31: 10k, Resistor_SMD:R_0805_2012Metric, F.Cu at (152.0, 18.3)
- added R62: 100R, Resistor_SMD:R_0805_2012Metric, F.Cu at (152.0, 21.2)
- added R63: 10k, Resistor_SMD:R_0805_2012Metric, F.Cu at (152.0, 24.2)
- added R64: 680R, Resistor_SMD:R_0805_2012Metric, F.Cu at (152.0, 27.1)
- added R94: 0R, Resistor_SMD:R_0805_2012Metric, F.Cu at (108.2, 45.9)
- added R95: 10k, Resistor_SMD:R_0805_2012Metric, F.Cu at (158.4, 18.3)
- added R96: 0R, Resistor_SMD:R_0805_2012Metric, F.Cu at (158.4, 21.2)
- added R97: 0R, Resistor_SMD:R_0805_2012Metric, F.Cu at (158.4, 24.2)
- added R98: 22R, Resistor_SMD:R_0805_2012Metric, F.Cu at (158.4, 27.1)
- added TP17: TestPoint, TestPoint:TestPoint_Pad_D1.5mm, F.Cu at (107.7, 35.3)
- added TP18: TestPoint, TestPoint:TestPoint_Pad_D1.5mm, F.Cu at (107.7, 38.9)
- added U19: MX25L1606EM1I-12G, Package_SO:SOP-8_3.76x4.96mm_P1.27mm, F.Cu at (164.9, 20.2)
Connections:
- net /AFE/SIPM_BIAS renamed /SiPMBiasRegulator/SIPM_BIAS_REG
- C39 pad 1: VCC -> /AnalogPowerNegative/VIN
- C40 pad 1: VCC -> /AnalogPowerNegative/VIN
- C41 pad 1: VCC -> /AnalogPowerNegative/VIN
- C52 pad 1: VCC -> /AnalogPowerNegative/VIN
- C53 pad 1: VCC -> /AnalogPowerNegative/VIN
- C62 pad 1: VCC -> /AnalogPowerNegative/VIN
- C65 pad 1: VCC -> /AnalogPowerNegative/VIN
- C78 pad 1: VCC -> /AnalogPowerNegative/VIN
- C82 pad 2: VCC -> /AnalogPowerNegative/VIN
- C85 pad 2: VCC -> /AnalogPowerNegative/VIN
- JP5 pad 1: VCC -> /AnalogPowerNegative/VIN
- JP6 pad 1: VCC -> /AnalogPowerNegative/VIN
- JP7 pad 1: VCC -> /AnalogPowerNegative/VIN
- JP8 pad 1: VCC -> /AnalogPowerNegative/VIN
- R13 pad 1: /SiPMBiasRegulator/SIPM_EN -> /FPGA/SIPM_EN
- R32 pad 2: VCC -> /AnalogPowerNegative/VIN
- R56 pad 2: VCC -> /AnalogPowerNegative/VIN
- R67 pad 1: VCC -> /AnalogPowerNegative/VIN
- R69 pad 1: VCC -> /AnalogPowerNegative/VIN
- R77 pad 1: VCC -> /AnalogPowerNegative/VIN
- R78 pad 2: VCC -> /AnalogPowerNegative/VIN
- R80 pad 1: VCC -> /AnalogPowerNegative/VIN
- R88 pad 2: VCC -> /AnalogPowerNegative/VIN
- U11 pad 1: VCC -> /AnalogPowerNegative/VIN
- U12 pad 1: VCC -> /AnalogPowerNegative/VIN
- U14 pad 1: VCC -> /AnalogPowerNegative/VIN
- U14 pad 2: VCC -> /AnalogPowerNegative/VIN
- U14 pad 3: VCC -> /AnalogPowerNegative/VIN
- U15 pad 1: VCC -> /AnalogPowerNegative/VIN
- U15 pad 2: VCC -> /AnalogPowerNegative/VIN
- U15 pad 3: VCC -> /AnalogPowerNegative/VIN
- U17 pad 1: VCC -> /AnalogPowerNegative/VIN
- U6 pad 100: Net-(U6B-VCCIO_1-Pad100) -> /ADC/VCC_3V3
- U6 pad 103: Net-(U6E-GND-Pad103) -> GND
- U6 pad 108: unconnected-(U6E-VPP_2V5-Pad108) -> /FPGA/VCC_2V5
- U6 pad 110: unconnected-(U6A-IOT_168-Pad110) -> /ADC/SIPM_ADC1
- U6 pad 111: Net-(U6E-VCC-Pad111) -> /ADC/VCC_3V3
- U6 pad 112: unconnected-(U6A-IOT_169-Pad112) -> /ADC/SIPM_ADC2
- U6 pad 113: unconnected-(U6A-IOT_170-Pad113) -> /ADC/SIPM_ADC3
- U6 pad 114: unconnected-(U6A-IOT_171-Pad114) -> /ADC/SIPM_ADC4
- U6 pad 115: unconnected-(U6A-IOT_172-Pad115) -> /ADC/SIPM_ADC5
- U6 pad 116: unconnected-(U6A-IOT_173-Pad116) -> /ADC/SIPM_ADC6
- U6 pad 117: unconnected-(U6A-IOT_174-Pad117) -> /ADC/SIPM_ADC7
- U6 pad 118: unconnected-(U6A-IOT_177-Pad118) -> /ADC/SIPM_ADC8
- U6 pad 119: unconnected-(U6A-IOT_178-Pad119) -> /ADC/SIPM_ADC9
- U6 pad 120: unconnected-(U6A-IOT_179-Pad120) -> /ADC/SIPM_ADC10
- U6 pad 121: unconnected-(U6A-IOT_181-Pad121) -> /ADC/SIPM_ADC11
- U6 pad 122: unconnected-(U6A-IOT_190-Pad122) -> /ADC/SIPM_ADC12
- U6 pad 123: Net-(U6A-VCCIO_0-Pad123) -> /ADC/VCC_3V3
- U6 pad 124: unconnected-(U6A-IOT_191-Pad124) -> /ADC/OTR
- U6 pad 125: unconnected-(U6A-IOT_192-Pad125) -> /FPGA/SIPM_EN
- U6 pad 126: unconnected-(U6E-VCCPLL1-Pad126) -> /DigitalPower/VCC_1V2
- U6 pad 127: unconnected-(U6E-GNDPLL1-Pad127) -> GND
- U6 pad 128: unconnected-(U6A-IOT_197_GBIN1-Pad128) -> /FPGA/SIPM_OVERLIGHT_FAULT
- U6 pad 13: Net-(U6E-GND-Pad103) -> GND
- U6 pad 131: Net-(U6A-VCCIO_0-Pad123) -> /ADC/VCC_3V3
- U6 pad 132: Net-(U6E-GND-Pad103) -> GND
- U6 pad 14: Net-(U6E-GND-Pad103) -> GND
- U6 pad 140: Net-(U6E-GND-Pad103) -> GND
- U6 pad 144: unconnected-(U6A-IOT_222-Pad144) -> Net-(U6A-IOT_222)
- U6 pad 27: Net-(U6E-VCC-Pad111) -> /ADC/VCC_3V3
- U6 pad 30: Net-(U6D-VCCIO_3-Pad30) -> /ADC/VCC_3V3
- U6 pad 40: Net-(U6E-VCC-Pad111) -> /ADC/VCC_3V3
- U6 pad 46: Net-(U6C-VCCIO_2-Pad46) -> /ADC/VCC_3V3
- U6 pad 5: Net-(U6E-GND-Pad103) -> GND
- U6 pad 53: unconnected-(U6E-GNDPLL0-Pad53) -> GND
- U6 pad 54: unconnected-(U6E-VCCPLL0-Pad54) -> /DigitalPower/VCC_1V2
- U6 pad 57: Net-(U6C-VCCIO_2-Pad46) -> /ADC/VCC_3V3
- U6 pad 59: Net-(U6E-GND-Pad103) -> GND
- U6 pad 6: Net-(U6D-VCCIO_3-Pad30) -> /ADC/VCC_3V3
- U6 pad 65: unconnected-(U6E-CDONE-Pad65) -> Net-(U6E-CDONE)
- U6 pad 66: unconnected-(U6E-~{CRESET}-Pad66) -> Net-(U6E-~{CRESET})
- U6 pad 67: unconnected-(U6E-IOB_105_SDO-Pad67) -> /FPGA/CFG_SPI_MOSI
- U6 pad 68: unconnected-(U6E-IOB_106_SDI-Pad68) -> /FPGA/CFG_SPI_MISO
- U6 pad 69: Net-(U6E-GND-Pad103) -> GND
- U6 pad 70: unconnected-(U6E-IOB_107_SCK-Pad70) -> /FPGA/CFG_SPI_SCK
- U6 pad 71: unconnected-(U6E-IOB_108_SS-Pad71) -> /FPGA/CFG_SPI_CS
- U6 pad 72: unconnected-(U6E-VCC_SPI-Pad72) -> /ADC/VCC_3V3
- U6 pad 86: Net-(U6E-GND-Pad103) -> GND
- U6 pad 89: Net-(U6B-VCCIO_1-Pad100) -> /ADC/VCC_3V3
- U6 pad 92: Net-(U6E-VCC-Pad111) -> /ADC/VCC_3V3

Commit message: fix: #160, fix: #163, fix: #164
Parts:
- added C12: 100n, Capacitor_SMD:C_0805_2012Metric, F.Cu at (246.4, 78.8)
- added C19: 100n, Capacitor_SMD:C_0805_2012Metric, F.Cu at (143.2, 66.7)
- added C23: 10n, Capacitor_SMD:C_0805_2012Metric, F.Cu at (143.2, 69.7)
- added C25: 10u/60V, Capacitor_SMD:C_0805_2012Metric, F.Cu at (197.5, 68.6)
- added C26: 100n/60V, Capacitor_SMD:C_0805_2012Metric, F.Cu at (197.5, 71.6)
- added C27: TBD, Capacitor_SMD:C_0805_2012Metric, F.Cu at (197.5, 74.6)
- added C28: 100n, Capacitor_SMD:C_0805_2012Metric, F.Cu at (239.9, 68.6)
- added C29: 10n, Capacitor_SMD:C_0805_2012Metric, F.Cu at (197.5, 77.7)
- added C30: 10n, Capacitor_SMD:C_0805_2012Metric, F.Cu at (197.5, 80.7)
- added C31: 10n, Capacitor_SMD:C_0805_2012Metric, F.Cu at (197.5, 83.7)
- added C32: 10u/60V, Capacitor_SMD:C_0805_2012Metric, F.Cu at (197.5, 86.7)
- added C33: 100n/60V, Capacitor_SMD:C_0805_2012Metric, F.Cu at (197.5, 89.7)
- added C41: 470n, Capacitor_SMD:C_0805_2012Metric, F.Cu at (246.4, 68.6)
- added C45: 10p, Capacitor_SMD:C_0805_2012Metric, F.Cu at (215.1, 34.0)
- added C47: 10u, Capacitor_SMD:C_0805_2012Metric, F.Cu at (215.1, 37.0)
- added C48: 10u, Capacitor_SMD:C_0805_2012Metric, F.Cu at (215.1, 40.0)
- added C49: 10u, Capacitor_SMD:C_0805_2012Metric, F.Cu at (215.1, 43.0)
- added C50: 100n, Capacitor_SMD:C_0805_2012Metric, F.Cu at (215.1, 46.0)
- added C51: 100n, Capacitor_SMD:C_0805_2012Metric, F.Cu at (136.7, 66.7)
- added C51: 10n, Capacitor_SMD:C_0805_2012Metric, F.Cu at (246.4, 71.6)
- added C54: 100n, Capacitor_SMD:C_0805_2012Metric, F.Cu at (246.4, 81.8)
- added C65: 10u, Capacitor_SMD:C_0805_2012Metric, F.Cu at (215.1, 49.1)
- added C66: 10u, Capacitor_SMD:C_0805_2012Metric, F.Cu at (215.1, 52.1)
- added C67: 100n, Capacitor_SMD:C_0805_2012Metric, F.Cu at (219.6, 34.0)
- added C68: 1u, Capacitor_SMD:C_0805_2012Metric, F.Cu at (219.6, 37.0)
- added C69: 1u, Capacitor_SMD:C_0805_2012Metric, F.Cu at (219.6, 40.0)
- added C70: 4u7, Capacitor_SMD:C_0805_2012Metric, F.Cu at (219.6, 43.0)
- added C71: 4u7 X7R, Capacitor_SMD:C_0805_2012Metric, F.Cu at (219.6, 46.0)
- added C72: 10u/16v, Capacitor_SMD:C_0805_2012Metric, F.Cu at (219.6, 49.1)
- added C73: 4u7, Capacitor_SMD:C_0805_2012Metric, F.Cu at (219.6, 52.1)
- added C74: 10u/16v, Capacitor_SMD:C_0805_2012Metric, F.Cu at (224.0, 34.0)
- added C75: 4u7 X7R, Capacitor_SMD:C_0805_2012Metric, F.Cu at (224.0, 37.0)
- added C76: 4u7, Capacitor_SMD:C_0805_2012Metric, F.Cu at (224.0, 40.0)
- added C77: 4u7, Capacitor_SMD:C_0805_2012Metric, F.Cu at (224.0, 43.0)
- added C78: 10u, Capacitor_SMD:C_0805_2012Metric, F.Cu at (220.2, 68.6)
- added C79: 10u, Capacitor_SMD:C_0805_2012Metric, F.Cu at (220.2, 71.6)
- added C80: 100n, Capacitor_SMD:C_0805_2012Metric, F.Cu at (220.2, 74.6)
- added C81: 1u, Capacitor_SMD:C_0805_2012Metric, F.Cu at (224.6, 68.6)
- added C82: 10u/16v, Capacitor_SMD:C_0805_2012Metric, F.Cu at (230.5, 34.0)
- added C83: 4u7 X7R, Capacitor_SMD:C_0805_2012Metric, F.Cu at (230.5, 37.0)
- added C84: 10u/16v, Capacitor_SMD:C_0805_2012Metric, F.Cu at (230.5, 40.0)
- added C85: 10u/16v, Capacitor_SMD:C_0805_2012Metric, F.Cu at (230.5, 43.0)
- added C86: 4u7 X7R, Capacitor_SMD:C_0805_2012Metric, F.Cu at (230.5, 46.0)
- added C87: 10u/16v, Capacitor_SMD:C_0805_2012Metric, F.Cu at (230.5, 49.1)
- added C88: 10p, Capacitor_SMD:C_0805_2012Metric, F.Cu at (224.6, 71.6)
- added C89: 10u, Capacitor_SMD:C_0805_2012Metric, F.Cu at (224.6, 74.6)
- added C90: 10u, Capacitor_SMD:C_0805_2012Metric, F.Cu at (229.1, 68.6)
- added C91: 10u, Capacitor_SMD:C_0805_2012Metric, F.Cu at (229.1, 71.6)
- added C92: 100n, Capacitor_SMD:C_0805_2012Metric, F.Cu at (229.1, 74.6)
- added C96: 100n, Capacitor_SMD:C_0805_2012Metric, F.Cu at (136.7, 69.7)
- added D5: DFLS1100-7, Diode_SMD:D_PowerDI-123, F.Cu at (198.3, 57.9)
- added D5: DFLS1100-7, Diode_SMD:D_PowerDI-123, F.Cu at (145.6, 61.3)
- added D6: DFLS1100-7, Diode_SMD:D_PowerDI-123, F.Cu at (137.5, 61.3)
- added D6: DFLS1100-7, Diode_SMD:D_PowerDI-123, F.Cu at (224.5, 78.0)
- added R12: 0R, Resistor_SMD:R_0805_2012Metric, F.Cu at (201.9, 68.6)
- added R13: 0R, Resistor_SMD:R_0805_2012Metric, F.Cu at (201.9, 71.5)
- added R14: TBD, Resistor_SMD:R_0805_2012Metric, F.Cu at (201.9, 74.5)
- added R15: 0R, Resistor_SMD:R_0805_2012Metric, F.Cu at (235.5, 68.6)
- added R16: 10k, Resistor_SMD:R_0805_2012Metric, F.Cu at (201.9, 77.4)
- added R17: 2M, Resistor_SMD:R_0805_2012Metric, F.Cu at (201.9, 80.4)
- added R18: TBD, Resistor_SMD:R_0805_2012Metric, F.Cu at (235.5, 71.5)
- added R19: 220k, Resistor_SMD:R_0805_2012Metric, F.Cu at (201.9, 83.3)
- added R20: 33k, Resistor_SMD:R_0805_2012Metric, F.Cu at (201.9, 86.3)
- added R21: 10k, Resistor_SMD:R_0805_2012Metric, F.Cu at (201.9, 89.2)
- added R25: 68k1, Resistor_SMD:R_0805_2012Metric, F.Cu at (197.5, 34.0)
- added R26: 10k, Resistor_SMD:R_0805_2012Metric, F.Cu at (197.5, 36.9)
- added R27: 0R, Resistor_SMD:R_0805_2012Metric, F.Cu at (197.5, 39.9)
- added R28: TBD, Resistor_SMD:R_0805_2012Metric, F.Cu at (197.5, 42.8)
- added R29: TBD, Resistor_SMD:R_0805_2012Metric, F.Cu at (235.5, 74.5)
- added R32: 0R, Resistor_SMD:R_0805_2012Metric, F.Cu at (197.5, 45.8)
- added R33: 0R, Resistor_SMD:R_0805_2012Metric, F.Cu at (197.5, 48.7)
- added R34: TBD, Resistor_SMD:R_0805_2012Metric, F.Cu at (197.5, 51.7)
- added R35: TBD, Resistor_SMD:R_0805_2012Metric, F.Cu at (197.5, 54.6)
- added R36: 19k5, Resistor_SMD:R_0805_2012Metric, F.Cu at (201.9, 34.0)
- added R37: 27k9, Resistor_SMD:R_0805_2012Metric, F.Cu at (201.9, 36.9)
- added R38: TBD, Resistor_SMD:R_0805_2012Metric, F.Cu at (201.9, 39.9)
- added R39: 0R, Resistor_SMD:R_0805_2012Metric, F.Cu at (201.9, 42.8)
- added R40: TBD, Resistor_SMD:R_0805_2012Metric, F.Cu at (201.9, 45.8)
- added R41: 0R, Resistor_SMD:R_0805_2012Metric, F.Cu at (201.9, 48.7)
- added R42: 0R, Resistor_SMD:R_0805_2012Metric, F.Cu at (201.9, 51.7)
- added R43: TBD, Resistor_SMD:R_0805_2012Metric, F.Cu at (201.9, 54.6)
- added R44: 0R, Resistor_SMD:R_0805_2012Metric, F.Cu at (206.3, 34.0)
- added R45: TBD, Resistor_SMD:R_0805_2012Metric, F.Cu at (206.3, 36.9)
- added R46: 0R, Resistor_SMD:R_0805_2012Metric, F.Cu at (206.3, 39.9)
- added R47: TBD, Resistor_SMD:R_0805_2012Metric, F.Cu at (206.3, 42.8)
- added R48: TBD, Resistor_SMD:R_0805_2012Metric, F.Cu at (206.3, 45.8)
- added R49: 0R, Resistor_SMD:R_0805_2012Metric, F.Cu at (206.3, 48.7)
- added R50: 49k9, Resistor_SMD:R_0805_2012Metric, F.Cu at (206.3, 51.7)
- added R51: 0R, Resistor_SMD:R_0805_2012Metric, F.Cu at (206.3, 54.6)
- added R52: 19k5, Resistor_SMD:R_0805_2012Metric, F.Cu at (210.7, 34.0)
- added R53: TBD, Resistor_SMD:R_0805_2012Metric, F.Cu at (210.7, 36.9)
- added R54: TBD, Resistor_SMD:R_0805_2012Metric, F.Cu at (210.7, 39.9)
- added R55: 0R, Resistor_SMD:R_0805_2012Metric, F.Cu at (210.7, 42.8)
- added R56: 0R, Resistor_SMD:R_0805_2012Metric, F.Cu at (215.7, 68.6)
- added R57: 0R, Resistor_SMD:R_0805_2012Metric, F.Cu at (215.7, 71.5)
- added R58: 47k, Resistor_SMD:R_0805_2012Metric, F.Cu at (215.7, 74.5)
- added R59: 200k, Resistor_SMD:R_0805_2012Metric, F.Cu at (215.7, 77.4)
- added R60: 10k, Resistor_SMD:R_0805_2012Metric, F.Cu at (215.7, 80.4)
- added R61: 0R, Resistor_SMD:R_0805_2012Metric, F.Cu at (215.7, 83.3)
- added R65: TBD, Resistor_SMD:R_0805_2012Metric, F.Cu at (246.3, 86.8)
- added R66: TBD, Resistor_SMD:R_0805_2012Metric, F.Cu at (246.3, 89.7)
- added R67: 0R, Resistor_SMD:R_0805_2012Metric, F.Cu at (234.9, 34.0)
- added R68: TBD, Resistor_SMD:R_0805_2012Metric, F.Cu at (234.9, 36.9)
- added R69: TBD, Resistor_SMD:R_0805_2012Metric, F.Cu at (234.9, 39.9)
- added R70: TBD, Resistor_SMD:R_0805_2012Metric, F.Cu at (234.9, 42.8)
- added R71: 49k9, Resistor_SMD:R_0805_2012Metric, F.Cu at (234.9, 45.8)
- added R72: 0R, Resistor_SMD:R_0805_2012Metric, F.Cu at (234.9, 48.7)
- added R73: 1k24, Resistor_SMD:R_0805_2012Metric, F.Cu at (239.3, 34.0)
- added R74: 0R, Resistor_SMD:R_0805_2012Metric, F.Cu at (239.3, 36.9)
- added R75: TBD, Resistor_SMD:R_0805_2012Metric, F.Cu at (239.3, 39.9)
- added R76: TBD, Resistor_SMD:R_0805_2012Metric, F.Cu at (239.3, 42.8)
- added R77: 0R, Resistor_SMD:R_0805_2012Metric, F.Cu at (239.3, 45.8)
- added R78: 0R, Resistor_SMD:R_0805_2012Metric, F.Cu at (239.3, 48.7)
- added R79: TBD, Resistor_SMD:R_0805_2012Metric, F.Cu at (243.7, 34.0)
- added R80: TBD, Resistor_SMD:R_0805_2012Metric, F.Cu at (243.7, 36.9)
- added R81: TBD, Resistor_SMD:R_0805_2012Metric, F.Cu at (243.7, 39.9)
- added R82: 24k9, Resistor_SMD:R_0805_2012Metric, F.Cu at (243.7, 42.8)
- added R83: 0R, Resistor_SMD:R_0805_2012Metric, F.Cu at (243.7, 45.8)
- added R84: 1k24, Resistor_SMD:R_0805_2012Metric, F.Cu at (243.7, 48.7)
- added R85: 0R, Resistor_SMD:R_0805_2012Metric, F.Cu at (248.1, 34.0)
- added R86: TBD, Resistor_SMD:R_0805_2012Metric, F.Cu at (248.1, 36.9)
- added R87: TBD, Resistor_SMD:R_0805_2012Metric, F.Cu at (248.1, 39.9)
- added R88: 0R, Resistor_SMD:R_0805_2012Metric, F.Cu at (248.1, 42.8)
- added R89: TBD, Resistor_SMD:R_0805_2012Metric, F.Cu at (215.7, 86.3)
- added R90: TBD, Resistor_SMD:R_0805_2012Metric, F.Cu at (235.5, 77.4)
- added R91: TBD, Resistor_SMD:R_0805_2012Metric, F.Cu at (235.5, 80.4)
- added R99: TBD, Resistor_SMD:R_0805_2012Metric, F.Cu at (235.5, 83.3)
- added TP10: TestPoint, TestPoint:TestPoint_Pad_D1.5mm, F.Cu at (205.9, 72.4)
- added TP11: TestPoint, TestPoint:TestPoint_Pad_D1.5mm, F.Cu at (205.9, 76.0)
- added TP12: TestPoint, TestPoint:TestPoint_Pad_D1.5mm, F.Cu at (239.5, 71.9)
- added TP13: TestPoint, TestPoint:TestPoint_Pad_D1.5mm, F.Cu at (205.9, 79.5)
- added TP14: TestPoint, TestPoint:TestPoint_Pad_D1.5mm, F.Cu at (205.9, 83.1)
- added TP15: REF_OUT, TestPoint:TestPoint_Pad_D1.5mm, F.Cu at (250.4, 73.5)
- added TP25: TestPoint, TestPoint:TestPoint_Pad_D1.5mm, F.Cu at (222.0, 55.3)
- added TP26: TestPoint, TestPoint:TestPoint_Pad_D1.5mm, F.Cu at (222.0, 58.9)
- added TP27: TestPoint, TestPoint:TestPoint_Pad_D1.5mm, F.Cu at (219.7, 77.9)
- added TP28: TestPoint, TestPoint:TestPoint_Pad_D1.5mm, F.Cu at (219.7, 81.5)
- added TP6: TestPoint, TestPoint:TestPoint_Pad_D1.5mm, F.Cu at (235.1, 88.6)
- added TP9: TestPoint, TestPoint:TestPoint_Pad_D1.5mm, F.Cu at (205.9, 68.9)
- added U10: LT3093, Package_SO:MSOP-12-1EP_3x4.039mm_P0.65mm_EP1.651x2.845mm_ThermalVias, F.Cu at (216.5, 62.3)
- added U13: REF3220AMDBVREP, Package_TO_SOT_SMD:SOT-23-6, F.Cu at (251.2, 69.5)
- added U14: LT3042, Package_SO:MSOP-12-1EP_3x4.039mm_P0.65mm_EP1.651x2.845mm_ThermalVias, F.Cu at (236.3, 53.2)
- added U15: LT3042, Package_SO:MSOP-12-1EP_3x4.039mm_P0.65mm_EP1.651x2.845mm_ThermalVias, F.Cu at (236.3, 59.0)
- added U16: LT8330IS6, Package_TO_SOT_SMD:TSOT-23-6, F.Cu at (224.1, 82.2)
- added U5: TPS7A4901, Package_SO:Texas_DGN0008B_VSSOP-8-1EP_3x3mm_P0.65mm_EP2x3mm_Mask1.88x1.98mm_ThermalVias, F.Cu at (207.8, 87.2)
- added U8: LT8330IS6, Package_TO_SOT_SMD:TSOT-23-6, F.Cu at (197.8, 62.1)
- added U9: LT3093, Package_SO:MSOP-12-1EP_3x4.039mm_P0.65mm_EP1.651x2.845mm_ThermalVias, F.Cu at (216.5, 56.5)
- TP17: value TestPoint -> GND
- TP18: value TestPoint -> +V_IN
- U3: value ~ -> LTC6268IS6
- U4: value ~ -> AD8139
- moved U14 12.0 mm to (125.1, 54.0)
- moved JP8 12.0 mm to (121.8, 58.2)
- moved U17 12.0 mm to (118.0, 54.2)
- moved C62 12.0 mm to (116.7, 57.9)
- moved C63 12.0 mm to (116.7, 60.9)
Connections:
- net /ADC/NEG renamed /ADC/AFE_OUT_N
- net /ADC/POS renamed /ADC/AFE_OUT_P
- net /DigitalPower/VCC_1V2 renamed /Digital Power/+1V2_D
- net /FPGA/CFG_RESET renamed /FPGA Configuration/CFG_RESET
- net /FPGA/CFG_SPI_CS renamed /FPGA Configuration/CFG_SPI_CS
- net /FPGA/CFG_SPI_MISO renamed /FPGA Configuration/CFG_SPI_MISO
- net /FPGA/CFG_SPI_MOSI renamed /FPGA Configuration/CFG_SPI_MOSI
- net /FPGA/CFG_SPI_SCK renamed /FPGA Configuration/CFG_SPI_SCK
- net /FPGA/VCC_2V5 renamed /Digital Power/+2V5_D
- net Net-(U6E-CDONE) renamed /FPGA Configuration/CFG_DONE
- C1 pad 1: /ADC/ADC_REF -> /ADC/+2V048_VREF
- C10 pad 1: /ADC/VCC_3V3 -> /ADC/+3V3_ADC
- C11 pad 1: /ADC/VCC_5V -> /ADC/+5V0_ADC
- C12 pad 1: /AFE/VCC_5V -> /AFE/AFE_AVDD_5V0
- C13 pad 1: /AFE/VCC_2V5 -> /AFE/+2V5_AFE
- C14 pad 2: /AFE/VEE_2V5 -> /AFE/-2V5_AFE
- C15 pad 1: /AFE/VCC_2V5 -> /AFE/+2V5_AFE
- C16 pad 2: /AFE/VEE_2V5 -> /AFE/-2V5_AFE
- C18 pad 1: /AFE/VCC_5V -> /ADC/+5V0_ADC
- C22 pad 1: /AFE/VCC_5V -> /ADC/+5V0_ADC
- C34 pad 1: /ADC/VCC_3V3 -> /Digital Power/+3V3_D
- C36 pad 1: /ADC/VCC_3V3 -> /Digital Power/+3V3_D
- C37 pad 1: /ADC/VCC_3V3 -> /Digital Power/+3V3_D
- C38 pad 1: /ADC/VCC_3V3 -> /Digital Power/+3V3_D
- C39 pad 1: /AnalogPowerNegative/VIN -> /Analog Power/+V_IN
- C40 pad 1: /AnalogPowerNegative/VIN -> /Analog Power/+V_IN
- C44 pad 1: /ADC/VCC_3V3 -> /Digital Power/+3V3_D
- C46 pad 1: /ADC/VCC_3V3 -> /Digital Power/+3V3_D
- C52 pad 1: /AnalogPowerNegative/VIN -> /Analog Power/+V_IN
- C53 pad 1: /AnalogPowerNegative/VIN -> /Analog Power/+V_IN
- C56 pad 1: /ADC/VCC_3V3 -> /Digital Power/+3V3_D
- C58 pad 1: /ADC/VCC_3V3 -> /Digital Power/+3V3_D
- C6 pad 1: /ADC/VCC_5V -> /ADC/+5V0_ADC
- C62 pad 1: /AnalogPowerNegative/VIN -> /Analog Power/+V_IN
- C63 pad 1: /ClockGeneration/VCC_3V3_CLK -> /Clock Generation/+3V3_CLKGEN
- C64 pad 1: /ClockGeneration/VCC_3V3_CLK -> /Clock Generation/+3V3_CLKGEN
- C69 pad 2: Net-(D3-A) -> Net-(D5-A)
- C70 pad 2: /AFE/VEE_2V5 -> /AFE/AFE_AVSS_2V5
- C73 pad 2: /AFE/VEE_2V5 -> /AFE/AFE_AVSS_2V5
- C76 pad 2: /AFE/VEE_5V -> /AFE/AFE_AVSS_5V0
- C77 pad 2: /AFE/VEE_5V -> /AFE/AFE_AVSS_5V0
- C8 pad 1: /ADC/VCC_3V3 -> /ADC/+3V3_ADC
- C84 pad 2: /AFE/VCC_5V -> /AFE/AFE_AVDD_5V0
- C87 pad 2: /AFE/VCC_2V5 -> /AFE/AFE_AVDD_2V5
- C88 pad 1: Net-(D4-K) -> Net-(D6-K)
- C89 pad 1: Net-(D4-K) -> Net-(D6-K)
- C9 pad 1: /ADC/VCC_5V -> /ADC/+5V0_ADC
- C90 pad 1: Net-(D4-K) -> Net-(D6-K)
- C93 pad 1: /ClockGeneration/VCC_3V3_CLK -> /Clock Generation/+3V3_CLKGEN
- C94 pad 1: /ClockGeneration/VCC_3V3_CLK -> /Clock Generation/+3V3_CLKGEN
- C95 pad 1: /ClockGeneration/VCC_3V3_CLK -> /Clock Generation/+3V3_CLKGEN
- C98 pad 1: /ADC/VCC_3V3 -> /Digital Power/+3V3_D
- C99 pad 1: /ADC/VCC_3V3 -> /Digital Power/+3V3_D
- JP6 pad 1: /AnalogPowerNegative/VIN -> /Analog Power/+V_IN
- JP7 pad 1: /AnalogPowerNegative/VIN -> /Analog Power/+V_IN
- JP8 pad 1: /AnalogPowerNegative/VIN -> /Analog Power/+V_IN
- R18 pad 2: /AFE/VCC_2V5 -> /AFE/AFE_AVDD_2V5
- R3 pad 2: /ADC/VCC_5V -> /ADC/+5V0_ADC
- R31 pad 2: /ADC/VCC_3V3 -> /Digital Power/+3V3_D
- R35 pad 1: /AFE/VEE_2V5 -> /AFE/AFE_AVSS_2V5
- R54 pad 1: /AFE/VEE_5V -> /AFE/AFE_AVSS_5V0
- R61 pad 2: Net-(D4-K) -> Net-(D6-K)
- R63 pad 2: /ADC/VCC_3V3 -> /Digital Power/+3V3_D
- R75 pad 2: /AFE/VCC_5V -> /AFE/AFE_AVDD_5V0
- R86 pad 2: /AFE/VCC_2V5 -> /AFE/AFE_AVDD_2V5
- R95 pad 2: /ADC/VCC_3V3 -> /Digital Power/+3V3_D
- R96 pad 2: /ADC/VCC_3V3 -> /Digital Power/+3V3_D
- R97 pad 2: /ADC/VCC_3V3 -> /Digital Power/+3V3_D
- TP1 pad 1: /AFE/VCC_2V5 -> /AFE/+2V5_AFE
- TP18 pad 1: /AnalogPowerNegative/VIN -> /Analog Power/+V_IN
- TP2 pad 1: /AFE/VEE_2V5 -> /AFE/-2V5_AFE
- TP20 pad 1: /ADC/VCC_3V3 -> /Digital Power/+3V3_D
- TP27 pad 1: Net-(D4-K) -> Net-(D6-K)
- TP5 pad 1: /AFE/VCC_5V -> /ADC/+5V0_ADC
- U10 pad 10: /AFE/VEE_5V -> /AFE/AFE_AVSS_5V0
- U10 pad 11: /AFE/VEE_5V -> /AFE/AFE_AVSS_5V0
- U10 pad 12: /AFE/VEE_5V -> /AFE/AFE_AVSS_5V0
- U11 pad 1: /AnalogPowerNegative/VIN -> /Analog Power/+V_IN
- U11 pad 5: /ADC/VCC_3V3 -> /Digital Power/+3V3_D
- U12 pad 1: /AnalogPowerNegative/VIN -> /Analog Power/+V_IN
- U14 pad 10: /AFE/VCC_5V -> /AFE/AFE_AVDD_5V0
- U14 pad 11: /AFE/VCC_5V -> /AFE/AFE_AVDD_5V0
- U14 pad 12: /AFE/VCC_5V -> /AFE/AFE_AVDD_5V0
- U15 pad 10: /AFE/VCC_2V5 -> /AFE/AFE_AVDD_2V5
- U15 pad 11: /AFE/VCC_2V5 -> /AFE/AFE_AVDD_2V5
- U15 pad 12: /AFE/VCC_2V5 -> /AFE/AFE_AVDD_2V5
- U16 pad 1: Net-(D4-A) -> Net-(D6-A)
- U17 pad 1: /AnalogPowerNegative/VIN -> /Analog Power/+V_IN
- U17 pad 5: /ClockGeneration/VCC_3V3_CLK -> /Clock Generation/+3V3_CLKGEN
- U18 pad 2: Net-(U18-CLK_EN) -> Net-(JP3-C)
- U18 pad 6: /ClockGeneration/VCC_3V3_CLK -> /Clock Generation/+3V3_CLKGEN
- U19 pad 8: /ADC/VCC_3V3 -> /Digital Power/+3V3_D
- U2 pad 3: /AFE/VCC_5V -> /AFE/AFE_AVDD_5V0
- U2 pad 4: /AFE/VCC_5V -> /AFE/AFE_AVDD_5V0
- U3 pad 2: /AFE/VEE_2V5 -> /AFE/-2V5_AFE
- U3 pad 5: /AFE/VCC_2V5 -> /AFE/+2V5_AFE
- U3 pad 6: /AFE/VCC_2V5 -> /AFE/+2V5_AFE
- U4 pad 2: /ADC/ADC_REF -> /ADC/+2V048_VREF
- U4 pad 3: /AFE/VCC_5V -> /ADC/+5V0_ADC
- U4 pad 6: /AFE/VEE_5V -> /AFE/-5V0_AFE
- U6 pad 100: /ADC/VCC_3V3 -> /Digital Power/+3V3_D
- U6 pad 111: /ADC/VCC_3V3 -> /Digital Power/+3V3_D
- U6 pad 123: /ADC/VCC_3V3 -> /Digital Power/+3V3_D
- U6 pad 125: /FPGA/SIPM_EN -> /FPGA/SIPM_BIAS_OK
- U6 pad 128: /FPGA/SIPM_OVERLIGHT_FAULT -> /FPGA/SIPM_BIAS_I2C_SCL
- U6 pad 129: unconnected-(U6A-IOT_198_GBIN0-Pad129) -> /FPGA/SIPM_BIAS_I2C_SDA
- U6 pad 131: /ADC/VCC_3V3 -> /Digital Power/+3V3_D
- U6 pad 27: /ADC/VCC_3V3 -> /Digital Power/+3V3_D
- U6 pad 30: /ADC/VCC_3V3 -> /Digital Power/+3V3_D
- U6 pad 40: /ADC/VCC_3V3 -> /Digital Power/+3V3_D
- U6 pad 46: /ADC/VCC_3V3 -> /Digital Power/+3V3_D
- U6 pad 57: /ADC/VCC_3V3 -> /Digital Power/+3V3_D
- U6 pad 6: /ADC/VCC_3V3 -> /Digital Power/+3V3_D
- U6 pad 72: /ADC/VCC_3V3 -> /Digital Power/+3V3_D
- U6 pad 89: /ADC/VCC_3V3 -> /Digital Power/+3V3_D
- U6 pad 92: /ADC/VCC_3V3 -> /Digital Power/+3V3_D
- U7 pad 1: Net-(U7-E/D) -> Net-(JP2-B)
- U7 pad 6: /ClockGeneration/VCC_3V3_CLK -> /Clock Generation/+3V3_CLKGEN
- U9 pad 10: /AFE/VEE_2V5 -> /AFE/AFE_AVSS_2V5
- U9 pad 11: /AFE/VEE_2V5 -> /AFE/AFE_AVSS_2V5
- U9 pad 12: /AFE/VEE_2V5 -> /AFE/AFE_AVSS_2V5
Routing:
- added copper zone on B.Cu, net GNDD
- added copper zone on F.Cu, net GNDD
