File: Hardware/GammaSpectrometer.kicad_blocks/AFE single channel.kicad_block/AFE single channel.kicad_sch (KiCad schematic)
At the start: 30 parts, among them U2001 OPA690xDBV, U2002 AD8139

Commit message: fix: #170
Parts:
- U2002: symbol DataAcquisitionUnit:AD8139 -> GammaSpectrometer:AD8139
Changed lines of the file:
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@@
 	)
 	(symbol
-		(lib_id "DataAcquisitionUnit:AD8139")
+		(lib_id "GammaSpectrometer:AD8139")
 		(at 130.81 57.15 0)
 		(unit 1)
