File: 03_SubsystemDesign/ElectronicHardware/Hardware/AnalogPower.kicad_sch (KiCad schematic)
At the start: 0 parts

Commit message: pcb design work in progress
Parts:
- added C1404, C1405, C1406, C1407, C1408, C1409: C, Capacitor_SMD:C_0805_2012Metric, symbol Device:C
- added R1401, R1402, R1403, R1404, R1405, R1406, R1407, R1408, R1409, R1410, R1411, R1412, R1413, R1414, R1415, R1416, R1417, R1418, R1419, R1420, R1421, R1422: R, Resistor_SMD:R_0805_2012Metric, symbol Device:R
- added TP1403, TP1404: TestPoint, TestPoint:TestPoint_Pad_D1.0mm, symbol Connector:TestPoint
- added U1401, U1402: LT3042, Package_SO:MSOP-12-1EP_3x4.039mm_P0.65mm_EP1.651x2.845mm_ThermalVias, symbol GammaSpectrometer:LT3042
Connections:
- net +3V3_A: now also C1409.2, R1419.2, TP1404.1, U1402.10 (OUTS), U1402.11 (OUT), U1402.12 (OUT)
- net +V_IN: now also C1404.2, C1405.2, R1401.1, R1403.1, R1405.1, R1407.1, R1421.2, R1422.2, U1401.1 (IN), U1401.2 (IN), U1401.3 (IN), U1402.1 (IN), U1402.2 (IN), U1402.3 (IN)
- new net: R1415.1, U1402.6 (I_LIM)
- new net: R1415.2, R1416.1
- new net: R1411.2, R1412.1
- new net: R1401.2, R1402.1, U1401.4 (EN/UV)
- new net: C1406.2, R1409.1, U1401.8 (SET)
- new net: R1405.2, R1406.1, U1401.5 (PG)
- new net: R1407.2, R1408.1, U1402.5 (PG)
- new net: R1417.1, R1418.2, R1421.1, U1401.7 (PFGB)
- new net: R1419.1, R1420.2, R1422.1, U1402.7 (PFGB)
- new net: R1403.2, R1404.1, U1402.4 (EN/UV)
- new net: R1413.1, U1401.6 (I_LIM)
- new net: C1407.2, R1411.1, U1402.8 (SET)
- new net: R1413.2, R1414.1
- new net: R1409.2, R1410.1
- new net +5V0_A: C1408.2, R1417.2, TP1403.1, U1401.10 (OUTS), U1401.11 (OUT), U1401.12 (OUT)
- new net GND: C1404.1, C1405.1, C1406.1, C1407.1, C1408.1, C1409.1, R1402.2, R1404.2, R1406.2, R1408.2, R1410.2, R1412.2, R1414.2, R1416.2, R1418.1, R1420.1, U1401.9 (GND), U1402.9 (GND)
Other:
- removed sheet Analog Power Negative
- removed sheet Analog Power Positive
- note added: "HIGH QUALITY CAPS FOR SET PIN!!!"
- note added: "LT3042 calculation: Rset = abs(Vout) / 100uA Ilimit = 125mA*kOhm / Rilim For: for 60 mA: Rilim = 125 / 60 = 2.08k for 70 mA: Rilim = 125 / 70 = 1.79k for 100 mA: Rilim = 125 / 100 = 1.24k PG not used -> leave PG floating PGFB not used -> tie PGFB to IN EN/UV tied to IN for always-on operation"
- note added: "OUTS is a sensor pin. Should be connected close to the IC that is supplied by this stabilizer on the PCB."
- note removed: "Note: This sheet groups Analog Power generation and distribution for readability. Positive and negative rails are shown on separate subsheets."

Commit message: improve CAD folder structure and PCB
Parts:
- added C1410, C1411, C1412, C1413, C1414: C, Capacitor_SMD:C_0805_2012Metric, symbol Device:C
- added R1423, R1424, R1425, R1426, R1427, R1428, R1429, R1430, R1431, R1432, R1433: R, Resistor_SMD:R_0805_2012Metric, symbol Device:R
- added TP1405: TestPoint, TestPoint:TestPoint_Pad_D1.0mm, symbol Connector:TestPoint
- added U1403: LT3042, Package_SO:MSOP-12-1EP_3x4.039mm_P0.65mm_EP1.651x2.845mm_ThermalVias, symbol GammaSpectrometer:LT3042
Connections:
- net +V_IN: now also C1410.2, C1412.2, R1423.1, R1425.1, R1433.2, U1403.1 (IN), U1403.2 (IN), U1403.3 (IN)
- net GND: now also C1410.1, C1411.1, C1412.1, C1413.1, C1414.1, R1424.2, R1426.2, R1428.2, R1430.2, R1432.1, U1403.13 (GND), U1403.9 (GND)
- new net: R1423.2, R1424.1, U1403.4 (EN/UV)
- new net: R1425.2, R1426.1, U1403.5 (PG)
- new net: R1431.1, R1432.2, R1433.1, U1403.7 (PFGB)
- new net: C1411.2, C1414.2, R1431.2, TP1405.1, U1403.10 (OUTS), U1403.11 (OUT), U1403.12 (OUT)
- new net: R1429.2, R1430.1
- new net: C1413.2, R1427.1, U1403.8 (SET)
- new net: R1427.2, R1428.1
- new net: R1429.1, U1403.6 (I_LIM)
Other:
- moved on the sheet: C1404, C1406, C1408, R1401, R1402, R1405, R1406, R1409, R1410, R1413, R1414, R1417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
