File: 03_SubsystemDesign/ElectronicHardware/Hardware/GammaSpectrometer.kicad_pcb (KiCad board)
At the start: 4 copper layers, 100 x 100 mm, 277 parts, among them J1801 USB_B_Micro, J301 RFShield_TwoPieces, U1002 LT3042, U1101 REF3220AMDBVREP, U1201 MX25L1606EM1I-12G, U1301 XLH736065.000000I, U1302 5PB1102PGGK, U1601 TPS7A4901, U1801 CH340X, U2001 OPA690xDBV, U2002 AD8139, U201 AD9238, U2101 OPA690xDBV, U2102 AD8139, U401 MCP4725A0T-E/CH, U402 MCP3221, U501 LT8330IS6, U601 ICE40HX4K-TQ144, U802 LT3093, U803 LT8330IS6, U901 NCP163ASN330T1G (3v3), U902 AP2112K-3.3, U903 AP2112K-1.2, U904 AP2112K-2.5, U905 TPS62932

Commit message: fix: #232
Parts:
- removed C1002, C1006, C803: 10u/16v, Capacitor_SMD:C_0805_2012Metric
- removed C1004, C807: 4u7 X7R, Capacitor_SMD:C_0805_2012Metric
- removed C1101: 470n, Capacitor_SMD:C_0805_2012Metric
- removed C1102, C2004, C2005, C2010, C2011, C2015, C210, C2105, C2106, C2107, C2112, C2113, C406, C407: 10n, Capacitor_SMD:C_0805_2012Metric
- removed C1903, C206, C207, C401, C402, C701, C703, C804, C815, C816, C818: 10u, Capacitor_SMD:C_0805_2012Metric
- removed C1904, C2001, C2002, C2006, C2007, C2014, C204, C205, C208, C209, C2102, C2103, C2104, C2110, C2111, C404, C405, C702, C704, C805, C817: 100n, Capacitor_SMD:C_0805_2012Metric
- removed C2003, C2101: 33p, Capacitor_SMD:C_0805_2012Metric
- removed C2008, C2009, C2108, C2109: 1p, Capacitor_SMD:C_0805_2012Metric
- removed C2012, C2114: 22p, Capacitor_SMD:C_0805_2012Metric
- removed C2013, C2016, C2017, C2115, C2116, C2117, C403: TBD, Capacitor_SMD:C_0805_2012Metric
- removed C808, C809: 1u, Capacitor_SMD:C_0805_2012Metric
- removed C811, C813: 4u7, Capacitor_SMD:C_0805_2012Metric
- removed C814: 10p, Capacitor_SMD:C_0805_2012Metric
- removed D801: DFLS1100-7, Diode_SMD:D_PowerDI-123
- removed R1003, R1012, R1016, R1022, R810, R814, R818, R825, R828: 0R, Resistor_SMD:R_0805_2012Metric
- removed R1004, R1007, R1008, R1019, R1020, R401, R403, R808, R809, R811, R822, R823: TBD, Resistor_SMD:R_0805_2012Metric
- removed R1011: 24k9, Resistor_SMD:R_0805_2012Metric
- removed R1015: 1k24, Resistor_SMD:R_0805_2012Metric
- removed R2001, R2101, R827: 10k, Resistor_SMD:R_0805_2012Metric
- removed R701, R702: 2k2, Resistor_SMD:R_0805_2012Metric
- removed R703: 680R, Resistor_SMD:R_0805_2012Metric
- removed R815: 49k9, Resistor_SMD:R_0805_2012Metric
- removed R819: 19k5, Resistor_SMD:R_0805_2012Metric
- removed R826: 68k1, Resistor_SMD:R_0805_2012Metric
- removed RN2001, RN2002, RN2101, RN2102: 1k, Resistor_SMD:R_Array_Convex_4x0612
- removed RN2003, RN2004, RN2103, RN2104: 100R, Resistor_SMD:R_Array_Convex_4x0612
- removed TP1001, TP2001, TP2002, TP2003, TP2004, TP2005, TP2101, TP2102, TP2103, TP2104, TP2105, TP803: TestPoint, TestPoint:TestPoint_Pad_D1.0mm
- removed TP1101: REF_OUT, TestPoint:TestPoint_Pad_D1.0mm
- removed TP402: SIPM_VOFFSET, TestPoint:TestPoint_Pad_D1.0mm
- removed U1002: LT3042, Package_SO:MSOP-12-1EP_3x4.039mm_P0.65mm_EP1.651x2.845mm_ThermalVias
- removed U1101: REF3220AMDBVREP, Package_TO_SOT_SMD:SOT-23-6
- removed U1301: XLH736065.000000I, Oscillator:Oscillator_SMD_IDT_JS6-6_5.0x3.2mm_P1.27mm
- removed U1302: 5PB1102PGGK, Package_SO:TSSOP-8_3x3mm_P0.65mm
- removed U2001, U2101: OPA690xDBV, Package_TO_SOT_SMD:SOT-23-6
- removed U2002, U2102: AD8139, Package_SO:SOIC-8_5.3x5.3mm_P1.27mm
- removed U401: MCP4725A0T-E/CH, Package_TO_SOT_SMD:SOT-23-6
- removed U402: MCP3221, Package_TO_SOT_SMD:SOT-23-5
- removed U601: ICE40HX4K-TQ144, Package_QFP:TQFP-144_20x20mm_P0.5mm
- removed U803: LT8330IS6, Package_TO_SOT_SMD:TSOT-23-6
- added C103: 1u, Capacitor_SMD:C_0805_2012Metric, F.Cu at (-82.3, 233.4)
- added C104: 10n, Capacitor_SMD:C_0805_2012Metric, F.Cu at (-82.3, 236.4)
- added C107: 1u, Capacitor_SMD:C_0805_2012Metric, F.Cu at (-82.3, 239.4)
- added C108: 10n, Capacitor_SMD:C_0805_2012Metric, F.Cu at (-82.3, 242.5)
- added C1404: C, Capacitor_SMD:C_0805_2012Metric, F.Cu at (148.4, 160.0)
- added C1405: C, Capacitor_SMD:C_0805_2012Metric, F.Cu at (74.4, 159.3)
- added C1406: C, Capacitor_SMD:C_0805_2012Metric, F.Cu at (148.4, 166.1)
- added C1407: C, Capacitor_SMD:C_0805_2012Metric, F.Cu at (74.4, 165.3)
- added C1408: C, Capacitor_SMD:C_0805_2012Metric, F.Cu at (148.4, 172.1)
- added C1409: C, Capacitor_SMD:C_0805_2012Metric, F.Cu at (74.4, 171.4)
- added C1410: C, Capacitor_SMD:C_0805_2012Metric, F.Cu at (181.2, 30.7)
- added C1411: C, Capacitor_SMD:C_0805_2012Metric, F.Cu at (187.1, 31.4)
- added C1412: C, Capacitor_SMD:C_0805_2012Metric, F.Cu at (181.2, 28.6)
- added C1413: C, Capacitor_SMD:C_0805_2012Metric, F.Cu at (187.2, 36.0)
- added C1414: C, Capacitor_SMD:C_0805_2012Metric, F.Cu at (189.2, 31.4)
- added C1804: 1u, Capacitor_SMD:C_0805_2012Metric, F.Cu at (98.5, 180.0)
- added C1805: 100n, Capacitor_SMD:C_0805_2012Metric, F.Cu at (98.5, 183.0)
- added C1806: 10n, Capacitor_SMD:C_0805_2012Metric, F.Cu at (98.5, 186.0)
- added C1807: 1u, Capacitor_SMD:C_0805_2012Metric, F.Cu at (98.5, 189.0)
- added C1808: 100n, Capacitor_SMD:C_0805_2012Metric, F.Cu at (98.5, 192.0)
- added C1809: 10n, Capacitor_SMD:C_0805_2012Metric, F.Cu at (98.5, 195.0)
- added C211: 100n, Capacitor_SMD:C_0805_2012Metric, F.Cu at (184.3, 143.0)
- added C212: 100n, Capacitor_SMD:C_0805_2012Metric, F.Cu at (184.3, 146.0)
- added C213: 100n, Capacitor_SMD:C_0805_2012Metric, F.Cu at (184.3, 149.0)
- added C214: 100n, Capacitor_SMD:C_0805_2012Metric, F.Cu at (181.2, 127.1)
- added C215: 100n, Capacitor_SMD:C_0805_2012Metric, F.Cu at (188.8, 133.9)
- added C216: 100n, Capacitor_SMD:C_0805_2012Metric, F.Cu at (188.8, 137.0)
- added C217: 1u, Capacitor_SMD:C_0805_2012Metric, F.Cu at (188.8, 140.0)
- added C218: 1u, Capacitor_SMD:C_0805_2012Metric, F.Cu at (188.8, 143.0)
- added C219: 10u, Capacitor_SMD:C_0805_2012Metric, F.Cu at (188.8, 146.0)
- added C220: 10u, Capacitor_SMD:C_0805_2012Metric, F.Cu at (188.8, 149.0)
- added C221: 1u, Capacitor_SMD:C_0805_2012Metric, F.Cu at (185.6, 127.1)
- added C222: 1u, Capacitor_SMD:C_0805_2012Metric, F.Cu at (193.2, 133.9)
- added C224: 10u, Capacitor_SMD:C_0805_2012Metric, F.Cu at (193.2, 137.0)
- added C225: 100n, Capacitor_SMD:C_0805_2012Metric, F.Cu at (193.2, 140.0)
- added C226: 10u, Capacitor_SMD:C_0805_2012Metric, F.Cu at (193.2, 143.0)
- added C227: 100n, Capacitor_SMD:C_0805_2012Metric, F.Cu at (193.2, 146.0)
- added C228: 10u, Capacitor_SMD:C_0805_2012Metric, F.Cu at (193.2, 149.0)
- added C229: 100n, Capacitor_SMD:C_0805_2012Metric, F.Cu at (190.1, 127.1)
- added C230: 10u, Capacitor_SMD:C_0805_2012Metric, F.Cu at (197.7, 133.9)
- added C231: 100n, Capacitor_SMD:C_0805_2012Metric, F.Cu at (197.7, 137.0)
- added C232: 100n, Capacitor_SMD:C_0805_2012Metric, F.Cu at (197.7, 140.0)
- added C233: 100n, Capacitor_SMD:C_0805_2012Metric, F.Cu at (197.7, 143.0)
- added C234: 1u, Capacitor_SMD:C_0805_2012Metric, F.Cu at (197.7, 146.0)
- added C235: 100n, Capacitor_SMD:C_0805_2012Metric, F.Cu at (197.7, 149.0)
- added C301: 1u, Capacitor_SMD:C_0805_2012Metric, F.Cu at (191.3, 47.4)
- added C302: 100n, Capacitor_SMD:C_0805_2012Metric, F.Cu at (191.3, 50.4)
- added C303: 1u, Capacitor_SMD:C_0805_2012Metric, F.Cu at (191.3, 52.5)
- added C304: 100n, Capacitor_SMD:C_0805_2012Metric, F.Cu at (191.3, 56.4)
- added C408: C, Capacitor_SMD:C_0805_2012Metric, F.Cu at (181.4, 70.2)
- added C409: C, Capacitor_SMD:C_0805_2012Metric, F.Cu at (184.3, 70.8)
- added C410: 2n2, Capacitor_SMD:C_0805_2012Metric, F.Cu at (187.9, 63.9)
- added C411: 1u, Capacitor_SMD:C_0805_2012Metric, F.Cu at (191.9, 69.1)
- added C412: C, Capacitor_SMD:C_0805_2012Metric, F.Cu at (181.4, 75.3)
- added C413: 100n, Capacitor_SMD:C_0805_2012Metric, F.Cu at (191.9, 67.0)
- added C414: C, Capacitor_SMD:C_0805_2012Metric, F.Cu at (181.4, 73.2)
- added C415: 10n, Capacitor_SMD:C_0805_2012Metric, F.Cu at (191.9, 64.9)
- added C416: C, Capacitor_SMD:C_0805_2012Metric, F.Cu at (190.9, 81.1)
- added C417: C, Capacitor_SMD:C_0805_2012Metric, F.Cu at (184.9, 81.1)
- added C418: 1u, Capacitor_SMD:C_0805_2012Metric, F.Cu at (181.4, 77.3)
- added C419: 100n, Capacitor_SMD:C_0805_2012Metric, F.Cu at (181.4, 79.4)
- added C420: 150p, Capacitor_SMD:C_0805_2012Metric, F.Cu at (187.9, 86.3)
- added C421: 10n, Capacitor_SMD:C_0805_2012Metric, F.Cu at (181.4, 81.5)
- added C422: 100p, Capacitor_SMD:C_0805_2012Metric, F.Cu at (190.9, 88.5)
- added C423: 100p, Capacitor_SMD:C_0805_2012Metric, F.Cu at (187.9, 91.1)
- added C424: 100p, Capacitor_SMD:C_0805_2012Metric, F.Cu at (184.9, 88.5)
- added C510: C, Capacitor_SMD:C_0805_2012Metric, F.Cu at (166.0, 70.5)
- added C511: C, Capacitor_SMD:C_0805_2012Metric, F.Cu at (168.9, 71.1)
- added C512: 2n2, Capacitor_SMD:C_0805_2012Metric, F.Cu at (172.6, 64.2)
- added C513: 1u, Capacitor_SMD:C_0805_2012Metric, F.Cu at (176.5, 69.4)
- added C514: C, Capacitor_SMD:C_0805_2012Metric, F.Cu at (166.0, 75.6)
- added C515: 100n, Capacitor_SMD:C_0805_2012Metric, F.Cu at (176.5, 67.3)
- added C516: C, Capacitor_SMD:C_0805_2012Metric, F.Cu at (166.0, 73.5)
- added C517: C, Capacitor_SMD:C_0805_2012Metric, F.Cu at (175.5, 81.4)
- added C518: C, Capacitor_SMD:C_0805_2012Metric, F.Cu at (169.5, 81.4)
- added C521: 150p, Capacitor_SMD:C_0805_2012Metric, F.Cu at (172.5, 86.6)
- added C522: 100p, Capacitor_SMD:C_0805_2012Metric, F.Cu at (175.5, 88.8)
- added C523: 100p, Capacitor_SMD:C_0805_2012Metric, F.Cu at (172.5, 91.4)
- added C524: 100p, Capacitor_SMD:C_0805_2012Metric, F.Cu at (169.5, 88.8)
- added C525: 10n, Capacitor_SMD:C_0805_2012Metric, F.Cu at (176.5, 65.2)
- added C526: 1u, Capacitor_SMD:C_0805_2012Metric, F.Cu at (166.0, 77.6)
- added C527: 100n, Capacitor_SMD:C_0805_2012Metric, F.Cu at (166.0, 79.7)
- added C528: 10n, Capacitor_SMD:C_0805_2012Metric, F.Cu at (166.0, 81.8)
- added C802: 1u, Capacitor_SMD:C_0805_2012Metric, F.Cu at (109.4, 189.1)
- added R103: 510R, Resistor_SMD:R_0805_2012Metric, F.Cu at (-77.9, 233.4)
- added R1401: R, Resistor_SMD:R_0805_2012Metric, F.Cu at (152.9, 160.0)
- added R1402: R, Resistor_SMD:R_0805_2012Metric, F.Cu at (152.9, 162.9)
- added R1403: R, Resistor_SMD:R_0805_2012Metric, F.Cu at (78.9, 162.2)
- added R1404: R, Resistor_SMD:R_0805_2012Metric, F.Cu at (78.9, 165.1)
- added R1405: R, Resistor_SMD:R_0805_2012Metric, F.Cu at (152.9, 171.8)
- added R1406: R, Resistor_SMD:R_0805_2012Metric, F.Cu at (152.9, 174.8)
- added R1407: R, Resistor_SMD:R_0805_2012Metric, F.Cu at (83.3, 156.3)
- added R1408: R, Resistor_SMD:R_0805_2012Metric, F.Cu at (83.3, 159.2)
- added R1409: R, Resistor_SMD:R_0805_2012Metric, F.Cu at (157.3, 165.9)
- added R1410: R, Resistor_SMD:R_0805_2012Metric, F.Cu at (157.3, 168.8)
- added R1411: R, Resistor_SMD:R_0805_2012Metric, F.Cu at (83.3, 168.1)
- added R1412: R, Resistor_SMD:R_0805_2012Metric, F.Cu at (83.3, 171.0)
- added R1413: R, Resistor_SMD:R_0805_2012Metric, F.Cu at (161.7, 160.0)
- added R1414: R, Resistor_SMD:R_0805_2012Metric, F.Cu at (161.7, 162.9)
- added R1415: R, Resistor_SMD:R_0805_2012Metric, F.Cu at (87.7, 162.2)
- added R1416: R, Resistor_SMD:R_0805_2012Metric, F.Cu at (87.7, 165.1)
- added R1417: R, Resistor_SMD:R_0805_2012Metric, F.Cu at (161.7, 171.8)
- added R1418: R, Resistor_SMD:R_0805_2012Metric, F.Cu at (161.7, 174.8)
- added R1419: R, Resistor_SMD:R_0805_2012Metric, F.Cu at (92.1, 156.3)
- added R1420: R, Resistor_SMD:R_0805_2012Metric, F.Cu at (92.1, 159.2)
- added R1421: R, Resistor_SMD:R_0805_2012Metric, F.Cu at (166.1, 165.9)
- added R1422: R, Resistor_SMD:R_0805_2012Metric, F.Cu at (92.1, 165.1)
- added R1423: R, Resistor_SMD:R_0805_2012Metric, F.Cu at (177.7, 33.0)
- added R1424: R, Resistor_SMD:R_0805_2012Metric, F.Cu at (177.7, 31.0)
- added R1425: R, Resistor_SMD:R_0805_2012Metric, F.Cu at (177.7, 35.0)
- added R1426: R, Resistor_SMD:R_0805_2012Metric, F.Cu at (177.7, 37.0)
- added R1427: R, Resistor_SMD:R_0805_2012Metric, F.Cu at (189.4, 36.0)
- added R1428: R, Resistor_SMD:R_0805_2012Metric, F.Cu at (189.5, 39.5)
- added R1429: R, Resistor_SMD:R_0805_2012Metric, F.Cu at (180.7, 38.3)
- added R1430: R, Resistor_SMD:R_0805_2012Metric, F.Cu at (177.7, 39.2)
- added R1431: R, Resistor_SMD:R_0805_2012Metric, F.Cu at (183.6, 41.6)
- added R1432: R, Resistor_SMD:R_0805_2012Metric, F.Cu at (183.6, 39.6)
- added R1433: R, Resistor_SMD:R_0805_2012Metric, F.Cu at (183.6, 37.5)
- added R1802: 2k2, Resistor_SMD:R_0805_2012Metric, F.Cu at (-106.8, 271.6)
- added R1803: 2k2, Resistor_SMD:R_0805_2012Metric, F.Cu at (-106.8, 274.5)
- added R1901: 510R, Resistor_SMD:R_0805_2012Metric, F.Cu at (117.0, 193.4)
- added R1902: 100R, Resistor_SMD:R_0805_2012Metric, F.Cu at (117.0, 196.3)
- added R1903: 100R, Resistor_SMD:R_0805_2012Metric, F.Cu at (117.0, 199.3)
- added R206: 22R, Resistor_SMD:R_0805_2012Metric, F.Cu at (209.3, 117.9)
- added R207: 22R, Resistor_SMD:R_0805_2012Metric, F.Cu at (209.3, 120.8)
- added R208: 22R, Resistor_SMD:R_0805_2012Metric, F.Cu at (209.3, 123.8)
- added R209: 22R, Resistor_SMD:R_0805_2012Metric, F.Cu at (187.9, 105.0)
- added R210: 22R, Resistor_SMD:R_0805_2012Metric, F.Cu at (184.2, 107.8)
- added R211: 22R, Resistor_SMD:R_0805_2012Metric, F.Cu at (213.7, 109.0)
- added R212: 22R, Resistor_SMD:R_0805_2012Metric, F.Cu at (213.7, 112.0)
- added R213: 22R, Resistor_SMD:R_0805_2012Metric, F.Cu at (213.7, 114.9)
- added R214: 22R, Resistor_SMD:R_0805_2012Metric, F.Cu at (213.7, 117.9)
- added R215: 22R, Resistor_SMD:R_0805_2012Metric, F.Cu at (213.7, 120.8)
- added R216: 22R, Resistor_SMD:R_0805_2012Metric, F.Cu at (213.7, 123.8)
- added R217: 22R, Resistor_SMD:R_0805_2012Metric, F.Cu at (179.4, 107.8)
- added R218: 22R, Resistor_SMD:R_0805_2012Metric, F.Cu at (177.4, 107.8)
- added R219: 22R, Resistor_SMD:R_0805_2012Metric, F.Cu at (218.1, 109.0)
- added R220: 22R, Resistor_SMD:R_0805_2012Metric, F.Cu at (218.1, 112.0)
- added R221: 22R, Resistor_SMD:R_0805_2012Metric, F.Cu at (218.1, 114.9)
- added R222: 22R, Resistor_SMD:R_0805_2012Metric, F.Cu at (218.1, 117.9)
- added R223: 22R, Resistor_SMD:R_0805_2012Metric, F.Cu at (218.1, 120.8)
- added R224: 22R, Resistor_SMD:R_0805_2012Metric, F.Cu at (218.1, 123.8)
- added R225: 22R, Resistor_SMD:R_0805_2012Metric, F.Cu at (173.3, 101.6)
- added R226: 22R, Resistor_SMD:R_0805_2012Metric, F.Cu at (173.3, 99.6)
- added R227: 22R, Resistor_SMD:R_0805_2012Metric, F.Cu at (222.5, 109.0)
- added R228: 22R, Resistor_SMD:R_0805_2012Metric, F.Cu at (222.5, 112.0)
- added R404: 2k, Resistor_SMD:R_0805_2012Metric, F.Cu at (187.9, 65.9)
- added R508: 2k, Resistor_SMD:R_0805_2012Metric, F.Cu at (172.6, 66.2)
- added R802: 22R, Resistor_SMD:R_0805_2012Metric, F.Cu at (104.9, 182.9)
- added R803: 22R, Resistor_SMD:R_0805_2012Metric, F.Cu at (104.9, 185.9)
- added R806: 22R, Resistor_SMD:R_0805_2012Metric, F.Cu at (104.9, 194.7)
- added RN401: 1k, Resistor_SMD:R_Array_Convex_4x0612, F.Cu at (187.9, 71.9)
- added RN402: 620R, Resistor_SMD:R_Array_Convex_4x0612, F.Cu at (187.9, 80.9)
- added RN403: 100R, Resistor_SMD:R_Array_Convex_4x0612, F.Cu at (187.9, 83.9)
- added RN404: 100R, Resistor_SMD:R_Array_Convex_4x0612, F.Cu at (187.9, 88.7)
- added RN501: 1k, Resistor_SMD:R_Array_Convex_4x0612, F.Cu at (172.5, 72.2)
- added RN502: 620R, Resistor_SMD:R_Array_Convex_4x0612, F.Cu at (172.5, 81.2)
- added RN503: 100R, Resistor_SMD:R_Array_Convex_4x0612, F.Cu at (172.5, 84.2)
- added RN504: 100R, Resistor_SMD:R_Array_Convex_4x0612, F.Cu at (172.5, 89.0)
- added TP1403: TestPoint, TestPoint:TestPoint_Pad_D1.0mm, F.Cu at (159.5, 177.8)
- added TP1404: TestPoint, TestPoint:TestPoint_Pad_D1.0mm, F.Cu at (85.5, 177.1)
- added TP1405: TestPoint, TestPoint:TestPoint_Pad_D1.0mm, F.Cu at (191.3, 32.4)
- added TP201: TestPoint, TestPoint:TestPoint_Pad_D1.0mm, F.Cu at (180.5, 130.1)
- added TP403: TestPoint, TestPoint:TestPoint_Pad_D1.0mm, F.Cu at (191.5, 71.3)
- added TP404: TestPoint, TestPoint:TestPoint_Pad_D1.0mm, F.Cu at (190.9, 83.9)
- added TP405: TestPoint, TestPoint:TestPoint_Pad_D1.0mm, F.Cu at (184.9, 83.9)
- added TP406: TestPoint, TestPoint:TestPoint_Pad_D1.0mm, F.Cu at (190.9, 91.3)
- added TP407: TestPoint, TestPoint:TestPoint_Pad_D1.0mm, F.Cu at (184.9, 91.3)
- added TP503: TestPoint, TestPoint:TestPoint_Pad_D1.0mm, F.Cu at (176.1, 71.6)
- added TP504: TestPoint, TestPoint:TestPoint_Pad_D1.0mm, F.Cu at (175.5, 84.2)
- added TP505: TestPoint, TestPoint:TestPoint_Pad_D1.0mm, F.Cu at (169.5, 84.2)
- added TP506: TestPoint, TestPoint:TestPoint_Pad_D1.0mm, F.Cu at (175.5, 91.6)
- added TP507: TestPoint, TestPoint:TestPoint_Pad_D1.0mm, F.Cu at (169.5, 91.6)
- added U101: ICE40HX4K-TQ144, Package_QFP:TQFP-144_20x20mm_P0.5mm, F.Cu at (118.1, 107.5)
- added U1401: LT3042, Package_SO:MSOP-12-1EP_3x4.039mm_P0.65mm_EP1.651x2.845mm_ThermalVias, F.Cu at (154.3, 179.2)
- added U1402: LT3042, Package_SO:MSOP-12-1EP_3x4.039mm_P0.65mm_EP1.651x2.845mm_ThermalVias, F.Cu at (80.3, 181.3)
- added U1403: LT3042, Package_SO:MSOP-12-1EP_3x4.039mm_P0.65mm_EP1.651x2.845mm_ThermalVias, F.Cu at (182.9, 34.1)
- added U302: ISL21010CFH325Z-T7A, Package_TO_SOT_SMD:SOT-23, F.Cu at (189.2, 50.6)
- added U403: MICROFC-60035-SMT-TR1_SiPM, GammaSpectrometer:MICROFC-60035-SMT-TR1_SiPM, F.Cu at (171.6, 56.9)
- added U404: MICROFC-60035-SMT-TR1_SiPM, GammaSpectrometer:MICROFC-60035-SMT-TR1_SiPM, F.Cu at (180.4, 47.6)
- added U405: LTC6268xS6-10, Package_TO_SOT_SMD:TSOT-23-6, F.Cu at (187.9, 68.7)
- added U406: AD8139, Package_SO:SOIC-8_5.3x5.3mm_P1.27mm, F.Cu at (187.9, 76.3)
- added U502: LTC6268xS6-10, Package_TO_SOT_SMD:TSOT-23-6, F.Cu at (172.6, 69.0)
- added U503: AD8139, Package_SO:SOIC-8_5.3x5.3mm_P1.27mm, F.Cu at (172.5, 76.6)
- added U504: MICROFC-60035-SMT-TR1_SiPM, GammaSpectrometer:MICROFC-60035-SMT-TR1_SiPM, F.Cu at (170.8, 48.1)
- added U505: MICROFC-60035-SMT-TR1_SiPM, GammaSpectrometer:MICROFC-60035-SMT-TR1_SiPM, F.Cu at (180.4, 56.6)
- added U801: 511JCA40M0000BAG, Oscillator:Oscillator_SMD_IDT_JS6-6_5.0x3.2mm_P1.27mm, F.Cu at (-81.7, 249.2)
- C1201, C1202, C1203, C1801, C501, C502, C506, C507, C508: value 10u -> C
- C1204, C1205, C1206, C1207, C1208, C1209, C1402, C1403, C1802, C1803, C503, C509, C904, C905, C909, C910, C912, C914, C915, C916, C917, C918, C919, C920, C921, C922: value 100n -> C
- C1210, C1604, C1605, C1606: value 10n -> C
- C1601, C1607: value 10u/60V -> C
- C1602, C1608: value 100n/60V -> C
- C1603: value TBD -> C
- C1901: value 10u -> 100n
- C203: value 100n -> 10u
- C504, C901, C902, C903, C906, C907, C908, C911, C913: value 1u -> C
- C505: value 10p -> C
- C801: value 10u -> 1u
- D501: value DFLS1100-7 -> D_Schottky
- JP901: value DVCC_CLK_ON -> SolderJumper_3_Bridged12
- JP902: value 3V3_ON -> SolderJumper_3_Bridged12
- JP903, JP904, JP906: value 1V2_ON -> SolderJumper_3_Bridged12
- R1201, R1203, R1207, R1604, R1608, R1801, R506: value 10k -> R
- R1202: value 100R -> R
- R1204: value 22R -> R
- R1205, R1206, R1601, R1602, R501, R502, R507: value 0R -> R
- R1603, R402, R503, R901, R902, R903, R904, R905, R906, R907: value TBD -> R
- R1605: value 2M -> R
- R1606: value 220k -> R
- R1607: value 33k -> R
- R201, R202: value TBD -> 1R
- R203, R204, R205, R804: value TBD -> 22R
- R504: value 47k -> R
- R505: value 200k -> R
- R801, R805: value 0R -> 22R
- TP1401: value +V_IN -> TestPoint
- TP1402: value GND -> TestPoint
- TP401: value SIPM_TEMP -> TestPoint
- U1601: value TPS7A4901 -> TPS7A49
- U802: value LT3093 -> SI53340-B-GMR; footprint Package_SO:MSOP-12-1EP_3x4.039mm_P0.65mm_EP1.651x2.845mm_ThermalVias -> Package_DFN_QFN:QFN-16-1EP_3x3mm_P0.5mm_EP1.9x1.9mm
- moved C1301 381.7 mm to (-61.5, 223.8)
- moved C1302 381.7 mm to (-61.5, 226.8)
- moved C1303 381.7 mm to (-61.5, 229.8)
- moved C1304 381.7 mm to (-61.5, 232.8)
- moved C1801 381.7 mm to (-95.4, 304.1)
- moved C1802 381.7 mm to (-95.4, 307.1)
- moved C1803 381.7 mm to (-95.4, 310.1)
- moved C901 381.7 mm to (-88.2, 188.6)
- moved C902 381.7 mm to (-88.2, 191.6)
- moved C903 381.7 mm to (-88.2, 194.6)
- moved C904 381.7 mm to (-88.2, 197.6)
- moved C905 381.7 mm to (-88.2, 200.6)
- moved C906 381.7 mm to (-88.2, 203.7)
- moved C907 381.7 mm to (-83.8, 188.6)
- moved C908 381.7 mm to (-83.8, 191.6)
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Connections:
- net /ADC/+3V3_ADC renamed /ADC/+3V3_D
- net /FPGA IO Banks/SIPM_BIAS_OK renamed /SiPM Bias/SIPM_BIAS_OK
- C202 pad 1: Net-(C201-Pad2) -> Net-(JP202-B)
- C202 pad 2: Net-(C202-Pad2) -> GND
- C203 pad 1: Net-(C202-Pad2) -> Net-(JP203-B)
- C801 pad 1: /Analog Power/+V_IN -> /Clock Generation/+3V3_CLKGEN
- R201 pad 1: Net-(R201-Pad1) -> Net-(FB201-Pad1)
- R201 pad 2: /ADC/+5V0_ADC -> Net-(JP202-B)
- R202 pad 1: GND -> Net-(FB202-Pad1)
- R202 pad 2: Net-(R201-Pad1) -> Net-(JP203-B)
- R203 pad 1: GND -> /ADC/SIPM_ADC_CH1_DATA12
- R203 pad 2: unconnected-(R203-Pad2) -> Net-(U201A-D11_A)
- R204 pad 1: Net-(R204-Pad1) -> /ADC/SIPM_ADC_CH1_DATA11
- R204 pad 2: /ADC/+2V048_VREF -> Net-(U201A-D10_A)
- R205 pad 1: GND -> /ADC/SIPM_ADC_CH1_DATA10
- R205 pad 2: Net-(R204-Pad1) -> Net-(U201A-D9_A)
- R801 pad 1: Net-(U803-VIN) -> /Clock Generation/FPGA_CLK_B0_P
- R801 pad 2: /Analog Power/+V_IN -> Net-(U802-Q0)
- R804 pad 1: Net-(U802-EN/UV) -> /Clock Generation/FPGA_CLK_B1_N
- R804 pad 2: GND -> Net-(U802-Q1b)
- R805 pad 1: /Analog Power/Analog Power Negative/VSS_RAW -> /Clock Generation/ADC_CLK_P
- R805 pad 2: Net-(U802-EN/UV) -> Net-(U802-Q2)
- TP801 pad 1: Net-(C814-Pad1) -> Net-(U802-CLK_0)
- TP802 pad 1: /Analog Power/Analog Power Negative/VSS_RAW -> Net-(U802-CLK_0b)
- U201 pad 1: unconnected-(U201-AGND-Pad1) -> GND
- U201 pad 10: unconnected-(U201-REFT_B-Pad10) -> Net-(U201F-REFB_B)
- U201 pad 11: unconnected-(U201-REFT_B-Pad11) -> Net-(U201F-REFT_B)
- U201 pad 12: unconnected-(U201-AVDD-Pad12) -> Net-(C201-Pad2)
- U201 pad 13: unconnected-(U201-AGND-Pad13) -> GND
- U201 pad 14: unconnected-(U201-V_IN_+B-Pad14) -> /ADC/AFE_OUT_CH2_P
- U201 pad 15: unconnected-(U201-V_IN_-B-Pad15) -> /ADC/AFE_OUT_CH2_N
- U201 pad 16: unconnected-(U201-AGND-Pad16) -> GND
- U201 pad 17: (no net) -> Net-(C201-Pad2)
- U201 pad 19: unconnected-(U201-DCS-Pad19) -> /ADC/DFS
- U201 pad 2: unconnected-(U201-V_IN_+A-Pad2) -> /ADC/AFE_OUT_CH1_P
- U201 pad 20: unconnected-(U201-DFS-Pad20) -> /ADC/DCS
- U201 pad 21: unconnected-(U201-PDWN_B-Pad21) -> /ADC/PDWN_B
- U201 pad 22: unconnected-(U201-OEB_B-Pad22) -> /ADC/OEB_B
- U201 pad 25: unconnected-(U201-D0_B-Pad25) -> Net-(U201B-D0_B)
- U201 pad 26: unconnected-(U201-D1_B-Pad26) -> Net-(U201B-D1_B)
- U201 pad 27: unconnected-(U201-D2_B-Pad27) -> Net-(U201B-D2_B)
- U201 pad 28: unconnected-(U201-DRGND-Pad28) -> GND
- U201 pad 29: unconnected-(U201-DRVDD-Pad29) -> Net-(C214-Pad2)
- U201 pad 3: unconnected-(U201-V_IN_-A-Pad3) -> /ADC/AFE_OUT_CH1_N
- U201 pad 30: unconnected-(U201-D3_B-Pad30) -> Net-(U201B-D3_B)
- U201 pad 31: unconnected-(U201-D4_B-Pad31) -> Net-(U201B-D4_B)
- U201 pad 32: unconnected-(U201-D5_B-Pad32) -> Net-(U201B-D5_B)
- U201 pad 33: unconnected-(U201-D6_B-Pad33) -> Net-(U201B-D6_B)
- U201 pad 34: unconnected-(U201-D7_B-Pad34) -> Net-(U201B-D7_B)
- U201 pad 35: unconnected-(U201-D8_B-Pad35) -> Net-(U201B-D8_B)
- U201 pad 36: unconnected-(U201-D9_B-Pad36) -> Net-(U201B-D9_B)
- U201 pad 37: unconnected-(U201-D10_B-Pad37) -> Net-(U201B-D10_B)
- U201 pad 38: unconnected-(U201-D11_B-Pad38) -> Net-(U201B-D11_B)
- U201 pad 39: unconnected-(U201-OTR_B-Pad39) -> Net-(U201B-OTR_B)
- U201 pad 4: unconnected-(U201-AGND-Pad4) -> GND
- U201 pad 40: unconnected-(U201-DRGND-Pad40) -> GND
- U201 pad 41: unconnected-(U201-DRVDD-Pad41) -> Net-(C214-Pad2)
- U201 pad 44: unconnected-(U201-D0_A-Pad44) -> Net-(U201A-D0_A)
- U201 pad 45: unconnected-(U201-D1_A-Pad45) -> Net-(U201A-D1_A)
- U201 pad 46: unconnected-(U201-D2_A-Pad46) -> Net-(U201A-D2_A)
- U201 pad 47: unconnected-(U201-D3_A-Pad47) -> Net-(U201A-D3_A)
- U201 pad 48: unconnected-(U201-D4_A-Pad48) -> Net-(U201A-D4_A)
- U201 pad 49: unconnected-(U201-D5_A-Pad49) -> Net-(U201A-D5_A)
- U201 pad 5: unconnected-(U201-AVDD-Pad5) -> Net-(C201-Pad2)
- U201 pad 50: unconnected-(U201-D6_A-Pad50) -> Net-(U201A-D6_A)
- U201 pad 51: unconnected-(U201-D7_A-Pad51) -> Net-(U201A-D7_A)
- U201 pad 52: unconnected-(U201-DRVDD-Pad52) -> Net-(C214-Pad2)
- U201 pad 53: unconnected-(U201-DRGND-Pad53) -> GND
- U201 pad 54: unconnected-(U201-D8_A-Pad54) -> Net-(U201A-D8_A)
- U201 pad 55: unconnected-(U201-D9_A-Pad55) -> Net-(U201A-D9_A)
- U201 pad 56: unconnected-(U201-D10_A-Pad56) -> Net-(U201A-D10_A)
- U201 pad 57: unconnected-(U201-D11_A-Pad57) -> Net-(U201A-D11_A)
- U201 pad 58: unconnected-(U201-OTR_A-Pad58) -> Net-(U201A-OTR_A)
- U201 pad 59: unconnected-(U201-OEB_A-Pad59) -> /ADC/OEB_A
- U201 pad 6: unconnected-(U201-REFT_A-Pad6) -> Net-(U201F-REFT_A)
- U201 pad 60: unconnected-(U201-PDWN_A-Pad60) -> /ADC/PDWN_A
- U201 pad 61: unconnected-(U201-MUX_SEL-Pad61) -> /ADC/MUX_SEL
- U201 pad 62: unconnected-(U201-SHR_REF-Pad62) -> Net-(JP204-C)
- U201 pad 64: unconnected-(U201-AVDD-Pad64) -> Net-(C201-Pad2)
- U201 pad 7: unconnected-(U201-REFB_A-Pad7) -> Net-(U201F-REFB_A)
- U201 pad 8: unconnected-(U201-VREF-Pad8) -> /ADC/+3V3_A
- U201 pad 9: unconnected-(U201-SENSE-Pad9) -> Net-(JP201-C)
- U802 pad 1: /Analog Power/Analog Power Negative/VSS_RAW -> GND
- U802 pad 10: /AFE/-5V0_AFE -> Net-(U802-Q0b)
- U802 pad 11: /AFE/-5V0_AFE -> Net-(U802-Q1)
- U802 pad 12: /AFE/-5V0_AFE -> Net-(U802-Q1b)
- U802 pad 13: /Analog Power/Analog Power Negative/VSS_RAW -> Net-(U802-Q2)
- U802 pad 2: /Analog Power/Analog Power Negative/VSS_RAW -> Net-(JP801-B)
- U802 pad 3: Net-(U802-EN/UV) -> Net-(U801-CLK+)
- U802 pad 5: Net-(U802-PFGB) -> /Clock Generation/+3V3_CLKGEN
- U802 pad 6: Net-(U802-I_LIM) -> Net-(U802-CLK_0)
- U802 pad 7: unconnected-(U802-VIOC-Pad7) -> Net-(U802-CLK_0b)
- U802 pad 8: Net-(U802-SET) -> unconnected-(U802-NC-Pad8)
- U802 pad 9: GND -> Net-(U802-Q0)
Routing:
- net (no net): track 176.3 -> 12.6 mm, vias 0 -> 2
- net /ADC/+5V0_ADC: track 151.5 -> 0.00 mm, vias 9 -> 0
- net /AFE/-5V0_AFE: track 139.5 -> 0.00 mm, vias 7 -> 0
- net Net-(RN2001-R3.2): track 49.6 -> 0.00 mm
- net Net-(U403-A): track 0.00 -> 39.2 mm
- net Net-(RN2001-R1.2): track 35.7 -> 0.00 mm
- net Net-(U1403-OUTS): track 0.00 -> 33.9 mm, vias 0 -> 2
- net /ADC/AFE_OUT_CH1_P: track 0.00 -> 27.4 mm
- net /ADC/AFE_OUT_CH2_P: track 0.00 -> 23.0 mm
- net Net-(RN2003-R3.1): track 22.4 -> 0.00 mm
- net Net-(RN2003-R1.1): track 22.4 -> 0.00 mm
- net /ADC/AFE_OUT_CH2_N: track 0.00 -> 20.8 mm
- net /AFE/+5V0_A: track 0.00 -> 15.7 mm, vias 0 -> 8
- net Net-(RN2101-R3.2): track 13.2 -> 0.00 mm
- net Net-(RN2101-R1.2): track 12.4 -> 0.00 mm
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- added copper zone on F.Cu, net (none)
- added copper zone on F.Cu, net /AFE/+5V0_A
- added copper zone on In1.Cu, net /AFE/+5V0_A
- added copper zone on F.Cu, net /AFE/AFEChannel1/1V5_REF
- added copper zone on F.Cu, net /Analog Power/+V_IN
- added copper zone on In1.Cu, net /Analog Power/+V_IN
- added copper zone on B.Cu, net GND
- added copper zone on F.Cu, net GND
- added copper zone on In2.Cu, net GND
- added copper zone on F.Cu, net Net-(U1403-EN/UV)
- removed copper zone on In1.Cu, net /ADC/+5V0_ADC
- removed copper zone on In1.Cu, net /AFE/-5V0_AFE

Commit message: add crystal holder to pcb
Parts:
- added U301: Untitled, GammaSpectrometer:ScintillatorCrystalHolder, F.Cu at (130.8, 49.3)
- moved U404 53.7 mm to (126.8, 45.0)
- moved U505 47.3 mm to (134.5, 45.0)
- moved U504 44.2 mm to (126.9, 53.5)
- moved U403 37.2 mm to (134.6, 53.5)
